Commit message: Updated CAD files for the Arm Simulation

File: kanga_arm/kanga_arm_description_dep/urdf/kanga_arm.urdf (robot description, URDF)
Before this commit: robot kanga_arm, 7 links, 6 joints
Links:
- link link_0: mass 2 -> 5
- link link_1: mass 3 -> 5
- link link_2: mass 3 -> 5
- link link_3: mass 3 -> 5
- link link_4: mass 0.7 -> 5; geometry collision mesh filename=../meshes/link_4.obj; visual mesh filename=../meshes/link_4.obj
- link link_5: mass 0.8 -> 10
Joints:
- joint J1: limit lower=-1.5708 upper=1.5708 effort=100 velocity=100 -> lower=-1.5708 upper=1.5708 effort=1000 velocity=1000
- joint J2: limit lower=-1.5708 upper=2.44346 effort=100 velocity=100 -> lower=-1.5708 upper=2.44346 effort=1000 velocity=1000; origin xyz=0.0855 -1.39264e-05 -0.056 rpy=-1.5708 9.90848e-17 1.5708 -> xyz=0.0855 -1.39264e-05 -0.056 rpy=-1.5708 -6.12323e-17 1.5708
- joint J3: limit lower=-1.8326 upper=2.87979 effort=100 velocity=100 -> lower=-1.8326 upper=2.87979 effort=1000 velocity=1000; origin xyz=-1.5984e-15 0.45 0.0405 rpy=9.42059e-16 3.67644e-15 -2.153e-15 -> xyz=2.76827e-16 0.45 0.0405 rpy=2.51629e-16 -8.53162e-16 -1.77023e-14
- joint J4: limit lower=-1.309 upper=2.35619 effort=100 velocity=100 -> lower=-1.309 upper=2.35619 effort=1000 velocity=1000; origin xyz=1.04906e-09 0.39 0.0525 rpy=1.18902e-15 8.86207e-15 1.5708 -> xyz=1.04906e-09 0.39 -0.015 rpy=-2.88523e-28 3.54659e-14 1.5708
- joint J5: limit lower=-1.5708 upper=1.5708 effort=100 velocity=100 -> lower=-1.5708 upper=1.5708 effort=1000 velocity=1000; origin xyz=0.03 1.6784e-14 -0.09644 rpy=3.14159 1.5708 0 -> xyz=0.105 3.43113e-14 -0.036 rpy=1.5708 3.82745e-33 -1.5708
- joint world_to_link_0: origin xyz=0 0 1.5 rpy=0 0 0 -> xyz=0 0 0.51 rpy=0 0 0
