Commit message: Working NavFN global with MPPI Local planner

File: kanga_sim/urdf/kanga_robot.urdf (robot description, URDF)
Before this commit: robot kangaSIM, 6 links, 5 joints
Links:
- link kangacore: geometry collision box size=0.489 0.72 0.35; visual mesh filename=file:///home/hunter/kanga/src/kanga_sim/urdf/kangacore.stl
- link wheel_a: geometry collision cylinder length=0.18 radius=0.125; visual mesh filename=file:///home/hunter/kanga/src/kanga_sim/urdf/wheel_a.stl
- link wheel_a_2: geometry collision cylinder length=0.18 radius=0.125; visual mesh filename=file:///home/hunter/kanga/src/kanga_sim/urdf/wheel_a.stl
- link wheelb: geometry collision cylinder length=0.18 radius=0.125; visual mesh filename=file:///home/hunter/kanga/src/kanga_sim/urdf/wheelb.stl
- link wheelb_2: geometry collision cylinder length=0.18 radius=0.125; visual mesh filename=file:///home/hunter/kanga/src/kanga_sim/urdf/wheelb.stl
Joints:
- joint base_link_to_kangacore: origin xyz=0.55486398 0.44572500 0.39697 rpy=0 0 1.5708 -> xyz=0.0 0.0 0.39697 rpy=0 0 1.5708
