Commit message: xacro implementation

File: kanga_description/urdf/assemblies/kanga_autonomous.urdf.xacro (robot description, xacro)
@@ -1,311 +1,11 @@
 <?xml version="1.0" ?>
-<robot name="kanga_autonomous">
-  <link name="base_link"/>
-  <joint name="base_link_to_kangacore" type="fixed">
-    <parent link="base_link"/>
-    <child link="kanga_core"/>
-    <!-- <origin xyz="0.55486398 0.44572500 0.39697" rpy="0 0 1.5708"/> -->
-    <origin xyz="0.0 0.0 0.39697" rpy="0 0 0"/>
-  </joint>
-  <!-- Link kanga_core -->
-  <link name="kanga_core">
-    <inertial>
-      <origin xyz="-0.0394422 -0.0149606 -0.0298892" rpy="0 0 0"/>
-      <mass value="28"/>
-      <inertia ixx="3.05326" ixy="-0.0953345" ixz="0.403632" iyy="4.37258" iyz="0.249778" izz="3.81615"/>
-    </inertial>
-    <!-- Part kangacore -->
-    <visual>
-      <origin xyz="-0.0406693 -0 0" rpy="0 -0 1.5708"/>
-      <geometry>
-        <mesh filename="package://kanga_description/meshes/core/kangacore.stl"/>
-      </geometry>
-      <material name="kangacore_material">
-        <color rgba="0.917647 0.917647 0.917647 1"/>
-      </material>
-    </visual>
-    <collision>
-      <origin xyz="-0.0406693 -0 0" rpy="0 -0 1.5708"/>
-      <geometry>
-        <mesh filename="package://kanga_description/meshes/core/kangacore.stl"/>
-      </geometry>
-    </collision>
-  </link>
-  <!-- Frame top_payload_mount (dummy link + fixed joint) -->
-  <link name="top_payload_mount">
-    <inertial>
-      <origin xyz="0 0 0" rpy="0 0 0"/>
-      <mass value="1e-9"/>
-      <inertia ixx="0" ixy="0" ixz="0" iyy="0" iyz="0" izz="0"/>
-    </inertial>
-  </link>
-  <joint name="top_payload_mount_frame" type="fixed">
-    <origin xyz="0.379844 -0.1575 0.1216" rpy="0 -0 0"/>
-    <parent link="kanga_core"/>
-    <child link="top_payload_mount"/>
-    <axis xyz="0 0 0"/>
-  </joint>
-  <!-- Frame front_payload_mount (dummy link + fixed joint) -->
-  <link name="front_payload_mount">
-    <inertial>
-      <origin xyz="0 0 0" rpy="0 0 0"/>
-      <mass value="1e-9"/>
-      <inertia ixx="0" ixy="0" ixz="0" iyy="0" iyz="0" izz="0"/>
-    </inertial>
-  </link>
-  <joint name="front_payload_mount_frame" type="fixed">
-    <origin xyz="0.158499 -0 0.0116" rpy="0 -0 0"/>
-    <parent link="kanga_core"/>
-    <child link="front_payload_mount"/>
-    <axis xyz="0 0 0"/>
-  </joint>
-  <!-- Link wheelb -->
-  <link name="wheelb">
-    <inertial>
-      <origin xyz="8.20141e-07 4.19108e-07 0.0294338" rpy="0 0 0"/>
-      <mass value="0.7"/>
-      <inertia ixx="0.00536519" ixy="2.6367e-08" ixz="3.55462e-07" iyy="0.00536521" iyz="7.378e-09" izz="0.00759451"/>
-    </inertial>
-    <!-- Part wheelb -->
-    <visual>
-      <origin xyz="0 0 -0.05" rpy="-1.5708 -0 0"/>
-      <geometry>
-        <mesh filename="package://kanga_description/meshes/core/wheelb.stl"/>
-      </geometry>
-      <material name="wheelb_material">
-        <color rgba="0.929412 0.0392157 0 1"/>
-      </material>
-    </visual>
-    <collision>
-      <origin xyz="0 0 -0.05" rpy="-1.5708 -0 0"/>
-      <geometry>
-        <mesh filename="package://kanga_description/meshes/core/wheelb.stl"/>
-      </geometry>
-    </collision>
-  </link>
-  <!-- Joint from kanga_core to wheelb -->
-  <joint name="wheel1" type="continuous">
-    <origin xyz="0.428413 0.395775 -0.271989" rpy="1.5708 0 0"/>
-    <parent link="kanga_core"/>
-    <child link="wheelb"/>
-    <axis xyz="0 0 1"/>
-    <limit effort="40" velocity="4.61"/>
-  </joint>
-  <!-- Link wheel_a -->
-  <link name="wheel_a">
-    <inertial>
-      <origin xyz="1.69548e-06 -4.25166e-07 0.0294802" rpy="0 0 0"/>
-      <mass value="0.7"/>
-      <inertia ixx="0.0053658" ixy="2.7862e-08" ixz="3.79976e-07" iyy="0.00536582" iyz="-5.263e-09" izz="0.00759416"/>
-    </inertial>
-    <!-- Part wheel_a -->
-    <visual>
-      <origin xyz="0 0 -0.05" rpy="-1.5708 0 0"/>
-      <geometry>
-        <mesh filename="package://kanga_description/meshes/core/wheel_a.stl"/>
-      </geometry>
-      <material name="wheel_a_material">
-        <color rgba="0.929412 0.0392157 0 1"/>
-      </material>
-    </visual>
-    <collision>
-      <origin xyz="0 0 -0.05" rpy="-1.5708 0 0"/>
-      <geometry>
-        <mesh filename="package://kanga_description/meshes/core/wheel_a.stl"/>
-      </geometry>
-    </collision>
-  </link>
-  <!-- Joint from kanga_core to wheel_a -->
-  <joint name="wheel2" type="continuous">
-    <origin xyz="-0.430143 0.395775 -0.272479" rpy="1.5708 0 -0"/>
-    <parent link="kanga_core"/>
-    <child link="wheel_a"/>
-    <axis xyz="0 0 1"/>
-    <limit effort="40" velocity="4.61"/>
-  </joint>
-  <!-- Link wheelb_2 -->
-  <link name="wheelb_2">
-    <inertial>
-      <origin xyz="8.20141e-07 4.19108e-07 0.0294338" rpy="0 0 0"/>
-      <mass value="0.7"/>
-      <inertia ixx="0.00536519" ixy="2.6367e-08" ixz="3.55462e-07" iyy="0.00536521" iyz="7.378e-09" izz="0.00759451"/>
-    </inertial>
-    <!-- Part wheelb_2 -->
-    <visual>
-      <origin xyz="0 0 -0.05" rpy="-1.5708 0 0"/>
-      <geometry>
-        <mesh filename="package://kanga_description/meshes/core/wheelb.stl"/>
-      </geometry>
-      <material name="wheelb_2_material">
-        <color rgba="0.929412 0.0392157 0 1"/>
-      </material>
-    </visual>
-    <collision>
-      <origin xyz="0 0 -0.05" rpy="-1.5708 0 0"/>
-      <geometry>
-        <mesh filename="package://kanga_description/meshes/core/wheelb.stl"/>
-      </geometry>
-    </collision>
-  </link>
-  <!-- Joint from kanga_core to wheelb_2 -->
-  <joint name="wheel3" type="continuous">
-    <origin xyz="-0.430143 -0.395725 -0.272479" rpy="1.5708 0 -3.14159"/>
-    <parent link="kanga_core"/>
-    <child link="wheelb_2"/>
-    <axis xyz="0 0 1"/>
-    <limit effort="40" velocity="4.61"/>
-  </joint>
-  <!-- Link wheel_a_2 -->
-  <link name="wheel_a_2">
-    <inertial>
-      <origin xyz="1.69548e-06 -4.25166e-07 0.0294802" rpy="0 0 0"/>
-      <mass value="0.7"/>
-      <inertia ixx="0.0053658" ixy="2.7862e-08" ixz="3.79976e-07" iyy="0.00536582" iyz="-5.263e-09" izz="0.00759416"/>
-    </inertial>
-    <!-- Part wheel_a_2 -->
-    <visual>
-      <origin xyz="0 0 -0.05" rpy="-1.5708 -0 0"/>
-      <geometry>
-        <mesh filename="package://kanga_description/meshes/core/wheel_a.stl"/>
-      </geometry>
-      <material name="wheel_a_2_material">
-        <color rgba="0.929412 0.0392157 0 1"/>
-      </material>
-    </visual>
-    <collision>
-      <origin xyz="0 0 -0.05" rpy="-1.5708 -0 0"/>
-      <geometry>
-        <mesh filename="package://kanga_description/meshes/core/wheel_a.stl"/>
-      </geometry>
-    </collision>
-  </link>
-  <!-- Joint from kanga_core to wheel_a_2 -->
-  <joint name="wheel4" type="continuous">
-    <origin xyz="0.428413 -0.395725 -0.271989" rpy="1.5708 -0 -3.14159"/>
-    <parent link="kanga_core"/>
-    <child link="wheel_a_2"/>
-    <axis xyz="0 0 1"/>
-    <limit effort="40" velocity="4.61"/>
-  </joint>
-  <!-- Attach autonomous lidar payload to the core top payload mount -->
-  <joint name="top_payload_mount_to_autonomous_lidar_payload" type="fixed">
-    <origin xyz="0 0 0" rpy="0 0 0"/>
-    <parent link="top_payload_mount"/>
-    <child link="autonomouslidarmount"/>
-    <axis xyz="0 0 0"/>
-  </joint>
-  <!-- Link autonomouslidarmount -->
-  <link name="autonomouslidarmount">
-    <inertial>
-      <origin xyz="-0.0301856 0.1375 0.184178" rpy="0 0 0"/>
-      <mass value="0.4"/>
-      <inertia ixx="0.0134847" ixy="3.8e-11" ixz="4.99203e-06" iyy="0.0100213" iyz="-2.9141e-08" izz="0.00357387"/>
-    </inertial>
-    <!-- Part autonomouslidarmount -->
-    <visual>
-      <origin xyz="-0.420514 0.1375 -0.1216" rpy="-0 -0 0"/>
-      <geometry>
-        <mesh filename="package://kanga_description/meshes/payloads/auto/autonomouslidarmount.stl"/>
-      </geometry>
-      <material name="autonomouslidarmount_material">
-        <color rgba="0.231373 0.380392 0.705882 1"/>
-      </material>
-    </visual>
-    <collision>
-      <origin xyz="-0.420514 0.1375 -0.1216" rpy="-0 -0 0"/>
-      <geometry>
-        <mesh filename="package://kanga_description/meshes/payloads/auto/autonomouslidarmount.stl"/>
-      </geometry>
-    </collision>
-  </link>
-  <!-- Frame UniLidarL2Mount (dummy link + fixed joint) -->
-  <link name="UniLidarL2Mount">
-    <origin xyz="0 0 0" rpy="0 -0 0"/>
-    <inertial>
-      <origin xyz="0 0 0" rpy="0 0 0"/>
-      <mass value="1e-9"/>
-      <inertia ixx="0" ixy="0" ixz="0" iyy="0" iyz="0" izz="0"/>
-    </inertial>
-  </link>
-  <joint name="UniLidarL2Mount_frame" type="fixed">
-    <origin xyz="-0.0300581 0.1375 0.355979" rpy="2.79253 -0 1.5708"/>
-    <parent link="autonomouslidarmount"/>
-    <child link="UniLidarL2Mount"/>
-    <axis xyz="0 0 0"/>
-  </joint>
-  <!-- UniLidarL2 attachment -->
-  <joint name="UniLidarL2_to_mount" type="fixed">
-    <origin xyz="0 0 0" rpy="0 0 0"/>
-    <parent link="UniLidarL2Mount"/>
-    <child link="unilidarl2base"/>
-    <axis xyz="0 0 0"/>
-  </joint>
-  <!-- Link unilidarl2base -->
-  <link name="unilidarl2base">
-    <inertial>
-      <origin xyz="-4.86924e-06 6.88756e-05 0.00436145" rpy="0 0 0"/>
-      <mass value="0.1"/>
-      <inertia ixx="4.60192e-05" ixy="-1.473e-09" ixz="-3.537e-09" iyy="4.63963e-05" iyz="9.141e-08" izz="8.42575e-05"/>
-    </inertial>
-    <visual>
-      <origin xyz="0.53025 -1.94934e-06 0.313234" rpy="3.14159 -0.349066 -3.14159"/>
-      <geometry>
-        <mesh filename="package://kanga_description/meshes/sensors/unilidar_l2/unilidarl2base.stl"/>
-      </geometry>
-      <material name="unilidarl2base_material">
-        <color rgba="0.301961 0.301961 0.301961 1"/>
-      </material>
-    </visual>
-    <collision>
-      <origin xyz="0.53025 -1.94934e-06 0.313234" rpy="3.14159 -0.349066 -3.14159"/>
-      <geometry>
-        <mesh filename="package://kanga_description/meshes/sensors/unilidar_l2/unilidarl2base.stl"/>
-      </geometry>
-    </collision>
-  </link>
-  <!-- Frame LidarBase (dummy link + fixed joint) -->
-  <link name="LidarBase">
-    <inertial>
-      <origin xyz="0 0 0" rpy="0 0 0"/>
-      <mass value="1e-9"/>
-      <inertia ixx="0" ixy="0" ixz="0" iyy="0" iyz="0" izz="0"/>
-    </inertial>
-  </link>
-  <joint name="LidarBase_frame" type="fixed">
-    <origin xyz="0 0 -0" rpy="0 0 1.5708"/>
-    <parent link="unilidarl2base"/>
-    <child link="LidarBase"/>
-    <axis xyz="0 0 0"/>
-  </joint>
-  <!-- Link unilidarl2top -->
-  <link name="unilidarl2top">
-    <inertial>
-      <origin xyz="-2.7414e-06 6.66489e-05 -0.0157604" rpy="0 0 0"/>
-      <mass value="0.13"/>
-      <inertia ixx="5.78833e-05" ixy="-1.075e-09" ixz="2.975e-09" iyy="3.66094e-05" iyz="9.3857e-08" izz="7.00661e-05"/>
-    </inertial>
-    <visual>
-      <origin xyz="-0.53025 -1.94934e-06 -0.290634" rpy="-0 0.349066 -0"/>
-      <geometry>
-        <mesh filename="package://kanga_description/meshes/sensors/unilidar_l2/unilidarl2top.stl"/>
-      </geometry>
-      <material name="unilidarl2top_material">
-        <color rgba="0.215686 0.215686 0.215686 1"/>
-      </material>
-    </visual>
-    <collision>
-      <origin xyz="-0.53025 -1.94934e-06 -0.290634" rpy="-0 0.349066 -0"/>
-      <geometry>
-        <mesh filename="package://kanga_description/meshes/sensors/unilidar_l2/unilidarl2top.stl"/>
-      </geometry>
-    </collision>
-  </link>
-  <!-- Joint from unilidarl2base to unilidarl2top -->
-  <joint name="LidarTop" type="revolute">
-    <origin xyz="0 0 0.0226" rpy="3.14159 -0 -3.14159"/>
-    <parent link="unilidarl2base"/>
-    <child link="unilidarl2top"/>
-    <axis xyz="0 0 1"/>
-    <limit effort="10" velocity="10" lower="0" upper="0"/>
-  </joint>
+<robot name="kanga_autonomous" xmlns:xacro="http://www.ros.org/wiki/xacro">
+  <!-- Top-level assembly:
+       combine base rover core + autonomous lidar payload. -->
+  <xacro:include filename="$(find kanga_description)/urdf/core/kanga_core_macro.urdf.xacro"/>
+  <xacro:include filename="$(find kanga_description)/urdf/payloads/autonomous/autonomous_lidar_payload_macro.urdf.xacro"/>
+  <!-- Build the rover base model first. -->
+  <xacro:kanga_core/>
+  <!-- Mount autonomous payload onto the core's top payload mount frame. -->
+  <xacro:autonomous_lidar_payload parent="top_payload_mount"/>
 </robot>

File: kanga_description/urdf/core/kanga_core.urdf.xacro (robot description, xacro)
@@ -1,192 +1,7 @@
 <?xml version="1.0" ?>
-<!-- Generated using onshape-to-robot -->
-<!-- Onshape https://tronsoc.onshape.com/documents/1c492049a2e71feeba4bb134/w/b322db97232ca622375ccdbf/e/3271415db943d39f5acebee7 -->
-<robot name="kanga_core">
-  <link name="base_link"/>
-  <joint name="base_link_to_kangacore" type="fixed">
-    <parent link="base_link"/>
-    <child link="kanga_core"/>
-    <!-- <origin xyz="0.55486398 0.44572500 0.39697" rpy="0 0 1.5708"/> -->
-    <origin xyz="0.0 0.0 0.39697" rpy="0 0 0"/>
-  </joint>
-  <!-- Link kanga_core -->
-  <link name="kanga_core">
-    <inertial>
-      <origin xyz="-0.0394422 -0.0149606 -0.0298892" rpy="0 0 0"/>
-      <mass value="28"/>
-      <inertia ixx="3.05326" ixy="-0.0953345" ixz="0.403632" iyy="4.37258" iyz="0.249778" izz="3.81615"/>
-    </inertial>
-    <!-- Part kangacore -->
-    <visual>
-      <origin xyz="-0.0406693 -0 0" rpy="0 -0 1.5708"/>
-      <geometry>
-        <mesh filename="package://kanga_description/meshes/core/kangacore.stl"/>
-      </geometry>
-      <material name="kangacore_material">
-        <color rgba="0.917647 0.917647 0.917647 1"/>
-      </material>
-    </visual>
-    <collision>
-      <origin xyz="-0.0406693 -0 0" rpy="0 -0 1.5708"/>
-      <geometry>
-        <mesh filename="package://kanga_description/meshes/core/kangacore.stl"/>
-      </geometry>
-    </collision>
-  </link>
-  <!-- Frame top_payload_mount (dummy link + fixed joint) -->
-  <link name="top_payload_mount">
-    <inertial>
-      <origin xyz="0 0 0" rpy="0 0 0"/>
-      <mass value="1e-9"/>
-      <inertia ixx="0" ixy="0" ixz="0" iyy="0" iyz="0" izz="0"/>
-    </inertial>
-  </link>
-  <joint name="top_payload_mount_frame" type="fixed">
-    <origin xyz="0.379844 -0.1575 0.1216" rpy="0 -0 0"/>
-    <parent link="kanga_core"/>
-    <child link="top_payload_mount"/>
-    <axis xyz="0 0 0"/>
-  </joint>
-  <!-- Frame front_payload_mount (dummy link + fixed joint) -->
-  <link name="front_payload_mount">
-    <inertial>
-      <origin xyz="0 0 0" rpy="0 0 0"/>
-      <mass value="1e-9"/>
-      <inertia ixx="0" ixy="0" ixz="0" iyy="0" iyz="0" izz="0"/>
-    </inertial>
-  </link>
-  <joint name="front_payload_mount_frame" type="fixed">
-    <origin xyz="0.158499 -0 0.0116" rpy="0 -0 0"/>
-    <parent link="kanga_core"/>
-    <child link="front_payload_mount"/>
-    <axis xyz="0 0 0"/>
-  </joint>
-  <!-- Link wheelb -->
-  <link name="wheelb">
-    <inertial>
-      <origin xyz="8.20141e-07 4.19108e-07 0.0294338" rpy="0 0 0"/>
-      <mass value="0.7"/>
-      <inertia ixx="0.00536519" ixy="2.6367e-08" ixz="3.55462e-07" iyy="0.00536521" iyz="7.378e-09" izz="0.00759451"/>
-    </inertial>
-    <!-- Part wheelb -->
-    <visual>
-      <origin xyz="0 0 -0.05" rpy="-1.5708 -0 0"/>
-      <geometry>
-        <mesh filename="package://kanga_description/meshes/core/wheelb.stl"/>
-      </geometry>
-      <material name="wheelb_material">
-        <color rgba="0.929412 0.0392157 0 1"/>
-      </material>
-    </visual>
-    <collision>
-      <origin xyz="0 0 -0.05" rpy="-1.5708 -0 0"/>
-      <geometry>
-        <mesh filename="package://kanga_description/meshes/core/wheelb.stl"/>
-      </geometry>
-    </collision>
-  </link>
-  <!-- Joint from kanga_core to wheelb -->
-  <joint name="wheel1" type="continuous">
-    <origin xyz="0.428413 0.395775 -0.271989" rpy="1.5708 0 0"/>
-    <parent link="kanga_core"/>
-    <child link="wheelb"/>
-    <axis xyz="0 0 1"/>
-    <limit effort="40" velocity="4.61"/>
-  </joint>
-  <!-- Link wheel_a -->
-  <link name="wheel_a">
-    <inertial>
-      <origin xyz="1.69548e-06 -4.25166e-07 0.0294802" rpy="0 0 0"/>
-      <mass value="0.7"/>
-      <inertia ixx="0.0053658" ixy="2.7862e-08" ixz="3.79976e-07" iyy="0.00536582" iyz="-5.263e-09" izz="0.00759416"/>
-    </inertial>
-    <!-- Part wheel_a -->
-    <visual>
-      <origin xyz="0 0 -0.05" rpy="-1.5708 0 0"/>
-      <geometry>
-        <mesh filename="package://kanga_description/meshes/core/wheel_a.stl"/>
-      </geometry>
-      <material name="wheel_a_material">
-        <color rgba="0.929412 0.0392157 0 1"/>
-      </material>
-    </visual>
-    <collision>
-      <origin xyz="0 0 -0.05" rpy="-1.5708 0 0"/>
-      <geometry>
-        <mesh filename="package://kanga_description/meshes/core/wheel_a.stl"/>
-      </geometry>
-    </collision>
-  </link>
-  <!-- Joint from kanga_core to wheel_a -->
-  <joint name="wheel2" type="continuous">
-    <origin xyz="-0.430143 0.395775 -0.272479" rpy="1.5708 0 -0"/>
-    <parent link="kanga_core"/>
-    <child link="wheel_a"/>
-    <axis xyz="0 0 1"/>
-    <limit effort="40" velocity="4.61"/>
-  </joint>
-  <!-- Link wheelb_2 -->
-  <link name="wheelb_2">
-    <inertial>
-      <origin xyz="8.20141e-07 4.19108e-07 0.0294338" rpy="0 0 0"/>
-      <mass value="0.7"/>
-      <inertia ixx="0.00536519" ixy="2.6367e-08" ixz="3.55462e-07" iyy="0.00536521" iyz="7.378e-09" izz="0.00759451"/>
-    </inertial>
-    <!-- Part wheelb_2 -->
-    <visual>
-      <origin xyz="0 0 -0.05" rpy="-1.5708 0 0"/>
-      <geometry>
-        <mesh filename="package://kanga_description/meshes/core/wheelb.stl"/>
-      </geometry>
-      <material name="wheelb_2_material">
-        <color rgba="0.929412 0.0392157 0 1"/>
-      </material>
-    </visual>
-    <collision>
-      <origin xyz="0 0 -0.05" rpy="-1.5708 0 0"/>
-      <geometry>
-        <mesh filename="package://kanga_description/meshes/core/wheelb.stl"/>
-      </geometry>
-    </collision>
-  </link>
-  <!-- Joint from kanga_core to wheelb_2 -->
-  <joint name="wheel3" type="continuous">
-    <origin xyz="-0.430143 -0.395725 -0.272479" rpy="1.5708 0 -3.14159"/>
-    <parent link="kanga_core"/>
-    <child link="wheelb_2"/>
-    <axis xyz="0 0 1"/>
-    <limit effort="40" velocity="4.61"/>
-  </joint>
-  <!-- Link wheel_a_2 -->
-  <link name="wheel_a_2">
-    <inertial>
-      <origin xyz="1.69548e-06 -4.25166e-07 0.0294802" rpy="0 0 0"/>
-      <mass value="0.7"/>
-      <inertia ixx="0.0053658" ixy="2.7862e-08" ixz="3.79976e-07" iyy="0.00536582" iyz="-5.263e-09" izz="0.00759416"/>
-    </inertial>
-    <!-- Part wheel_a_2 -->
-    <visual>
-      <origin xyz="0 0 -0.05" rpy="-1.5708 -0 0"/>
-      <geometry>
-        <mesh filename="package://kanga_description/meshes/core/wheel_a.stl"/>
-      </geometry>
-      <material name="wheel_a_2_material">
-        <color rgba="0.929412 0.0392157 0 1"/>
-      </material>
-    </visual>
-    <collision>
-      <origin xyz="0 0 -0.05" rpy="-1.5708 -0 0"/>
-      <geometry>
-        <mesh filename="package://kanga_description/meshes/core/wheel_a.stl"/>
-      </geometry>
-    </collision>
-  </link>
-  <!-- Joint from kanga_core to wheel_a_2 -->
-  <joint name="wheel4" type="continuous">
-    <origin xyz="0.428413 -0.395725 -0.271989" rpy="1.5708 -0 -3.14159"/>
-    <parent link="kanga_core"/>
-    <child link="wheel_a_2"/>
-    <axis xyz="0 0 1"/>
-    <limit effort="40" velocity="4.61"/>
-  </joint>
+<robot name="kanga_core" xmlns:xacro="http://www.ros.org/wiki/xacro">
+  <!-- Wrapper file:
+       include the reusable core macro and instantiate it as a standalone model. -->
+  <xacro:include filename="$(find kanga_description)/urdf/core/kanga_core_macro.urdf.xacro"/>
+  <xacro:kanga_core/>
 </robot>
