Commit message: xacro implementation

File: kanga_description/urdf/payloads/autonomous/autonomous_lidar_payload.urdf.xacro (robot description, xacro)
@@ -1,119 +1,10 @@
 <?xml version="1.0" ?>
-<!-- Generated using onshape-to-robot -->
-<!-- Onshape https://tronsoc.onshape.com/documents/a04fc62c100c90ae88802972/w/c0a63c4f09140e5b63a1ee94/e/6441c68a791f9e1842cd52ba -->
-<robot name="autonomous_lidar_payload">
-  <!-- Link autonomouslidarmount -->
-  <link name="autonomouslidarmount">
-    <inertial>
-      <origin xyz="-0.0301856 0.1375 0.184178" rpy="0 0 0"/>
-      <mass value="0.4"/>
-      <inertia ixx="0.0134847" ixy="3.8e-11" ixz="4.99203e-06" iyy="0.0100213" iyz="-2.9141e-08" izz="0.00357387"/>
-    </inertial>
-    <!-- Part autonomouslidarmount -->
-    <visual>
-      <origin xyz="-0.420514 0.1375 -0.1216" rpy="-0 -0 0"/>
-      <geometry>
-        <mesh filename="package://kanga_description/meshes/payloads/auto/autonomouslidarmount.stl"/>
-      </geometry>
-      <material name="autonomouslidarmount_material">
-        <color rgba="0.231373 0.380392 0.705882 1"/>
-      </material>
-    </visual>
-    <collision>
-      <origin xyz="-0.420514 0.1375 -0.1216" rpy="-0 -0 0"/>
-      <geometry>
-        <mesh filename="package://kanga_description/meshes/payloads/auto/autonomouslidarmount.stl"/>
-      </geometry>
-    </collision>
-  </link>
-  <!-- Frame UniLidarL2Mount (dummy link + fixed joint) -->
-  <link name="UniLidarL2Mount">
-    <origin xyz="0 0 0" rpy="0 -0 0"/>
-    <inertial>
-      <origin xyz="0 0 0" rpy="0 0 0"/>
-      <mass value="1e-9"/>
-      <inertia ixx="0" ixy="0" ixz="0" iyy="0" iyz="0" izz="0"/>
-    </inertial>
-  </link>
-  <joint name="UniLidarL2Mount_frame" type="fixed">
-    <origin xyz="-0.0300581 0.1375 0.355979" rpy="2.79253 -0 1.5708"/>
-    <parent link="autonomouslidarmount"/>
-    <child link="UniLidarL2Mount"/>
-    <axis xyz="0 0 0"/>
-  </joint>
-  <!-- UniLidarL2 attachment -->
-  <joint name="UniLidarL2_to_mount" type="fixed">
-    <origin xyz="0 0 0" rpy="0 0 0"/>
-    <parent link="UniLidarL2Mount"/>
-    <child link="unilidarl2base"/>
-    <axis xyz="0 0 0"/>
-  </joint>
-  <!-- Link unilidarl2base -->
-  <link name="unilidarl2base">
-    <inertial>
-      <origin xyz="-4.86924e-06 6.88756e-05 0.00436145" rpy="0 0 0"/>
-      <mass value="0.1"/>
-      <inertia ixx="4.60192e-05" ixy="-1.473e-09" ixz="-3.537e-09" iyy="4.63963e-05" iyz="9.141e-08" izz="8.42575e-05"/>
-    </inertial>
-    <visual>
-      <origin xyz="0.53025 -1.94934e-06 0.313234" rpy="3.14159 -0.349066 -3.14159"/>
-      <geometry>
-        <mesh filename="package://kanga_description/meshes/sensors/unilidar_l2/unilidarl2base.stl"/>
-      </geometry>
-      <material name="unilidarl2base_material">
-        <color rgba="0.301961 0.301961 0.301961 1"/>
-      </material>
-    </visual>
-    <collision>
-      <origin xyz="0.53025 -1.94934e-06 0.313234" rpy="3.14159 -0.349066 -3.14159"/>
-      <geometry>
-        <mesh filename="package://kanga_description/meshes/sensors/unilidar_l2/unilidarl2base.stl"/>
-      </geometry>
-    </collision>
-  </link>
-  <!-- Frame LidarBase (dummy link + fixed joint) -->
-  <link name="LidarBase">
-    <inertial>
-      <origin xyz="0 0 0" rpy="0 0 0"/>
-      <mass value="1e-9"/>
-      <inertia ixx="0" ixy="0" ixz="0" iyy="0" iyz="0" izz="0"/>
-    </inertial>
-  </link>
-  <joint name="LidarBase_frame" type="fixed">
-    <origin xyz="0 0 -0" rpy="0 0 1.5708"/>
-    <parent link="unilidarl2base"/>
-    <child link="LidarBase"/>
-    <axis xyz="0 0 0"/>
-  </joint>
-  <!-- Link unilidarl2top -->
-  <link name="unilidarl2top">
-    <inertial>
-      <origin xyz="-2.7414e-06 6.66489e-05 -0.0157604" rpy="0 0 0"/>
-      <mass value="0.13"/>
-      <inertia ixx="5.78833e-05" ixy="-1.075e-09" ixz="2.975e-09" iyy="3.66094e-05" iyz="9.3857e-08" izz="7.00661e-05"/>
-    </inertial>
-    <visual>
-      <origin xyz="-0.53025 -1.94934e-06 -0.290634" rpy="-0 0.349066 -0"/>
-      <geometry>
-        <mesh filename="package://kanga_description/meshes/sensors/unilidar_l2/unilidarl2top.stl"/>
-      </geometry>
-      <material name="unilidarl2top_material">
-        <color rgba="0.215686 0.215686 0.215686 1"/>
-      </material>
-    </visual>
-    <collision>
-      <origin xyz="-0.53025 -1.94934e-06 -0.290634" rpy="-0 0.349066 -0"/>
-      <geometry>
-        <mesh filename="package://kanga_description/meshes/sensors/unilidar_l2/unilidarl2top.stl"/>
-      </geometry>
-    </collision>
-  </link>
-  <!-- Joint from unilidarl2base to unilidarl2top -->
-  <joint name="LidarTop" type="revolute">
-    <origin xyz="0 0 0.0226" rpy="3.14159 -0 -3.14159"/>
-    <parent link="unilidarl2base"/>
-    <child link="unilidarl2top"/>
-    <axis xyz="0 0 1"/>
-    <limit effort="10" velocity="10" lower="0" upper="0"/>
-  </joint>
+<robot name="autonomous_lidar_payload" xmlns:xacro="http://www.ros.org/wiki/xacro">
+  <!-- Wrapper file:
+       Include the reusable autonomous payload macro and instantiate it standalone. -->
+  <xacro:include filename="$(find kanga_description)/urdf/payloads/autonomous/autonomous_lidar_payload_macro.urdf.xacro"/>
+  <!-- Local root used only when visualizing payload by itself. -->
+  <link name="base_link"/>
+  <!-- Instantiate payload and attach to local root. -->
+  <xacro:autonomous_lidar_payload parent="base_link"/>
 </robot>

File: kanga_description/urdf/sensors/UniLidarL2/UniLidarL2.urdf.xacro (robot description, xacro)
@@ -1,72 +1,10 @@
 <?xml version="1.0" ?>
-<!-- UniLidarL2 sensor model exported from Onshape and adapted for kanga_description meshes -->
-<robot name="UniLidarL2">
-  <!-- Link unilidarl2base -->
-  <link name="unilidarl2base">
-    <inertial>
-      <origin xyz="-4.86924e-06 6.88756e-05 0.00436145" rpy="0 0 0"/>
-      <mass value="0.1"/>
-      <inertia ixx="4.60192e-05" ixy="-1.473e-09" ixz="-3.537e-09" iyy="4.63963e-05" iyz="9.141e-08" izz="8.42575e-05"/>
-    </inertial>
-    <visual>
-      <origin xyz="0.53025 -1.94934e-06 0.313234" rpy="3.14159 -0.349066 -3.14159"/>
-      <geometry>
-        <mesh filename="package://kanga_description/meshes/sensors/unilidar_l2/unilidarl2base.stl"/>
-      </geometry>
-      <material name="unilidarl2base_material">
-        <color rgba="0.301961 0.301961 0.301961 1"/>
-      </material>
-    </visual>
-    <collision>
-      <origin xyz="0.53025 -1.94934e-06 0.313234" rpy="3.14159 -0.349066 -3.14159"/>
-      <geometry>
-        <mesh filename="package://kanga_description/meshes/sensors/unilidar_l2/unilidarl2base.stl"/>
-      </geometry>
-    </collision>
-  </link>
-  <!-- Frame LidarBase (dummy link + fixed joint) -->
-  <link name="LidarBase">
-    <inertial>
-      <origin xyz="0 0 0" rpy="0 0 0"/>
-      <mass value="1e-9"/>
-      <inertia ixx="0" ixy="0" ixz="0" iyy="0" iyz="0" izz="0"/>
-    </inertial>
-  </link>
-  <joint name="LidarBase_frame" type="fixed">
-    <origin xyz="0 0 -0" rpy="0 0 1.5708"/>
-    <parent link="unilidarl2base"/>
-    <child link="LidarBase"/>
-    <axis xyz="0 0 0"/>
-  </joint>
-  <!-- Link unilidarl2top -->
-  <link name="unilidarl2top">
-    <inertial>
-      <origin xyz="-2.7414e-06 6.66489e-05 -0.0157604" rpy="0 0 0"/>
-      <mass value="0.13"/>
-      <inertia ixx="5.78833e-05" ixy="-1.075e-09" ixz="2.975e-09" iyy="3.66094e-05" iyz="9.3857e-08" izz="7.00661e-05"/>
-    </inertial>
-    <visual>
-      <origin xyz="-0.53025 -1.94934e-06 -0.290634" rpy="-0 0.349066 -0"/>
-      <geometry>
-        <mesh filename="package://kanga_description/meshes/sensors/unilidar_l2/unilidarl2top.stl"/>
-      </geometry>
-      <material name="unilidarl2top_material">
-        <color rgba="0.215686 0.215686 0.215686 1"/>
-      </material>
-    </visual>
-    <collision>
-      <origin xyz="-0.53025 -1.94934e-06 -0.290634" rpy="-0 0.349066 -0"/>
-      <geometry>
-        <mesh filename="package://kanga_description/meshes/sensors/unilidar_l2/unilidarl2top.stl"/>
-      </geometry>
-    </collision>
-  </link>
-  <!-- Joint from unilidarl2base to unilidarl2top -->
-  <joint name="LidarTop" type="revolute">
-    <origin xyz="0 0 0.0226" rpy="3.14159 -0 -3.14159"/>
-    <parent link="unilidarl2base"/>
-    <child link="unilidarl2top"/>
-    <axis xyz="0 0 1"/>
-    <limit effort="10" velocity="10" lower="0" upper="0"/>
-  </joint>
+<robot name="UniLidarL2" xmlns:xacro="http://www.ros.org/wiki/xacro">
+  <!-- Wrapper file:
+       Include the reusable lidar macro and instantiate it as a standalone model. -->
+  <xacro:include filename="$(find kanga_description)/urdf/sensors/UniLidarL2/UniLidarL2_macro.urdf.xacro"/>
+  <!-- Local root used only when visualizing the lidar by itself. -->
+  <link name="base_link"/>
+  <!-- Instantiate the reusable macro and attach it to this root. -->
+  <xacro:unilidar_l2 parent="base_link"/>
 </robot>
