Commit message: Complete Xacro URDF for lidar mount

File: kanga_description/onshape_export/UniLidarL2/UniLidarL2.urdf (robot description, URDF)
Before this commit: robot UniLidarL2, 3 links, 2 joints
Links:
- removed link LidarBase
- link unilidarl2base: geometry collision mesh filename=package://kanga_description/assets_UniLidarL2/unilidarl2bas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; visual mesh filename=package://kanga_description/assets_UniLidarL2/unilidarl2bas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
- link unilidarl2top: geometry collision mesh filename=package://kanga_description/assets_UniLidarL2/unilidarl2top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; visual mesh filename=package://kanga_description/assets_UniLidarL2/unilidarl2top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
Joints:
- removed joint LidarBase_frame
- joint LidarTop: origin xyz=0 0 0.0226 rpy=3.14159 -0 -3.14159 -> xyz=-0 0 0.0214 rpy=0 -0 0

File: kanga_description/onshape_export/autonomous_lidar_payload/autonomous_lidar_payload.urdf (robot description, URDF)
Before this commit: robot autonomous_lidar_payload, 3 links, 2 joints
Links:
- removed link AutonomousLidarMount
- removed link UniLidarL2Mount
- added link autonomous_lidar_mount, mass 1e-9
- added link unilidarl2_mount, mass 1e-9
- link autonomouslidarmount: geometry collision mesh filename=package://kanga_description/assets_autonomous_lidar_payload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; visual mesh filename=package://kanga_description/assets_autonomous_lidar_payload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
Joints:
- removed joint AutonomousLidarMount_frame
- removed joint UniLidarL2Mount_frame
- added joint autonomous_lidar_mount_frame: type fixed, parent autonomouslidarmount, child autonomous_lidar_mount, origin xyz=0 0 0 rpy=0 -0 0, axis 0 0 0
- added joint unilidarl2_mount_frame: type fixed, parent autonomouslidarmount, child unilidarl2_mount, origin xyz=-0.0300581 0.1575 0.355979 rpy=2.79253 -0 1.5708, axis 0 0 0

File: kanga_description/urdf/core/kanga_core_macro.urdf.xacro (robot description, xacro)
@@ -65,6 +65,6 @@
   </joint>
   <!-- Drive wheel links and joints. -->
-  <!-- Link wheelb -->
-  <link name="wheelb">
+  <!-- Link wheel_FL -->
+  <link name="wheel_FL">
     <inertial>
       <origin xyz="8.20141e-07 4.19108e-07 0.0294338" rpy="0 0 0"/>
@@ -89,14 +89,14 @@
     </collision>
   </link>
-  <!-- Joint from kanga_core to wheelb -->
+  <!-- Joint from kanga_core to wheel_FL -->
   <joint name="wheel1" type="continuous">
     <origin xyz="0.428413 0.395775 -0.271989" rpy="1.5708 0 0"/>
     <parent link="kanga_core"/>
-    <child link="wheelb"/>
+    <child link="wheel_FL"/>
     <axis xyz="0 0 1"/>
     <limit effort="40" velocity="4.61"/>
   </joint>
-  <!-- Link wheel_a -->
-  <link name="wheel_a">
+  <!-- Link wheel_BL -->
+  <link name="wheel_BL">
     <inertial>
       <origin xyz="1.69548e-06 -4.25166e-07 0.0294802" rpy="0 0 0"/>
@@ -121,14 +121,14 @@
     </collision>
   </link>
-  <!-- Joint from kanga_core to wheel_a -->
+  <!-- Joint from kanga_core to wheel_BL -->
   <joint name="wheel2" type="continuous">
     <origin xyz="-0.430143 0.395775 -0.272479" rpy="1.5708 0 -0"/>
     <parent link="kanga_core"/>
-    <child link="wheel_a"/>
+    <child link="wheel_BL"/>
     <axis xyz="0 0 1"/>
     <limit effort="40" velocity="4.61"/>
   </joint>
-  <!-- Link wheelb_2 -->
-  <link name="wheelb_2">
+  <!-- Link wheel_BR -->
+  <link name="wheel_BR">
     <inertial>
       <origin xyz="8.20141e-07 4.19108e-07 0.0294338" rpy="0 0 0"/>
@@ -153,14 +153,14 @@
     </collision>
   </link>
-  <!-- Joint from kanga_core to wheelb_2 -->
+  <!-- Joint from kanga_core to wheel_BR -->
   <joint name="wheel3" type="continuous">
     <origin xyz="-0.430143 -0.395725 -0.272479" rpy="1.5708 0 -3.14159"/>
     <parent link="kanga_core"/>
-    <child link="wheelb_2"/>
+    <child link="wheel_BR"/>
     <axis xyz="0 0 1"/>
     <limit effort="40" velocity="4.61"/>
   </joint>
-  <!-- Link wheel_a_2 -->
-  <link name="wheel_a_2">
+  <!-- Link wheel_FR -->
+  <link name="wheel_FR">
     <inertial>
       <origin xyz="1.69548e-06 -4.25166e-07 0.0294802" rpy="0 0 0"/>
@@ -185,9 +185,9 @@
     </collision>
   </link>
-  <!-- Joint from kanga_core to wheel_a_2 -->
+  <!-- Joint from kanga_core to wheel_FR -->
   <joint name="wheel4" type="continuous">
     <origin xyz="0.428413 -0.395725 -0.271989" rpy="1.5708 -0 -3.14159"/>
     <parent link="kanga_core"/>
-    <child link="wheel_a_2"/>
+    <child link="wheel_FR"/>
     <axis xyz="0 0 1"/>
     <limit effort="40" velocity="4.61"/>

File: kanga_description/urdf/payloads/autonomous/autonomous_lidar_payload_macro.urdf.xacro (robot description, xacro)
@@ -19,19 +19,19 @@
     <link name="${prefix}autonomouslidarmount">
       <inertial>
-        <origin xyz="-0.0301856 0.1375 0.184178" rpy="0 0 0"/>
+        <origin xyz="-0.0301856 0.1575 0.184178" rpy="0 0 0"/>
         <mass value="0.4"/>
         <inertia ixx="0.0134847" ixy="3.8e-11" ixz="4.99203e-06" iyy="0.0100213" iyz="-2.9141e-08" izz="0.00357387"/>
       </inertial>
       <visual>
-        <origin xyz="-0.420514 0.1375 -0.1216" rpy="-0 -0 0"/>
+        <origin xyz="-0.420514 0.1575 -0.1216" rpy="-0 -0 0"/>
         <geometry>
           <mesh filename="package://kanga_description/meshes/payloads/auto/autonomouslidarmount.stl"/>
         </geometry>
         <material name="autonomouslidarmount_material">
-          <color rgba="0.231373 0.380392 0.705882 1"/>
+          <color rgba="0.5 0.5 0.5 1"/>
         </material>
       </visual>
       <collision>
-        <origin xyz="-0.420514 0.1375 -0.1216" rpy="-0 -0 0"/>
+        <origin xyz="-0.420514 0.1575 -0.1216" rpy="-0 -0 0"/>
         <geometry>
           <mesh filename="package://kanga_description/meshes/payloads/auto/autonomouslidarmount.stl"/>
@@ -48,5 +48,5 @@
     </link>
     <joint name="${prefix}UniLidarL2Mount_frame" type="fixed">
-      <origin xyz="-0.0300581 0.1375 0.355979" rpy="2.79253 -0 1.5708"/>
+      <origin xyz="-0.0300581 0.1575 0.355979" rpy="2.79253 -0 1.5708"/>
       <parent link="${prefix}autonomouslidarmount"/>
       <child link="${prefix}UniLidarL2Mount"/>

File: kanga_description/urdf/sensors/UniLidarL2/UniLidarL2_macro.urdf.xacro (robot description, xacro)
@@ -17,12 +17,12 @@
     <link name="${prefix}unilidarl2base">
       <inertial>
-        <origin xyz="-4.86924e-06 6.88756e-05 0.00436145" rpy="0 0 0"/>
+        <origin xyz="6.88756e-05 4.86924e-06 0.00436145" rpy="0 0 0"/>
         <mass value="0.1"/>
-        <inertia ixx="4.60192e-05" ixy="-1.473e-09" ixz="-3.537e-09" iyy="4.63963e-05" iyz="9.141e-08" izz="8.42575e-05"/>
+        <inertia ixx="4.63963e-05" ixy="1.473e-09" ixz="9.141e-08" iyy="4.60192e-05" iyz="3.537e-09" izz="8.42575e-05"/>
       </inertial>
       <visual>
-        <origin xyz="0.53025 -1.94934e-06 0.313234" rpy="3.14159 -0.349066 -3.14159"/>
+        <origin xyz="-1.94934e-06 -0.53025 0.313234" rpy="3.14159 -0.349066 1.5708"/>
         <geometry>
-          <mesh filename="package://kanga_description/meshes/sensors/unilidar_l2/unilidarl2base.stl"/>
+          <mesh filename="package://kanga_description/urdf/sensors/UniLidarL2/meshes/unilidarl2base.stl"/>
         </geometry>
         <material name="unilidarl2base_material">
@@ -31,35 +31,21 @@
       </visual>
       <collision>
-        <origin xyz="0.53025 -1.94934e-06 0.313234" rpy="3.14159 -0.349066 -3.14159"/>
+        <origin xyz="-1.94934e-06 -0.53025 0.313234" rpy="3.14159 -0.349066 1.5708"/>
         <geometry>
-          <mesh filename="package://kanga_description/meshes/sensors/unilidar_l2/unilidarl2base.stl"/>
+          <mesh filename="package://kanga_description/urdf/sensors/UniLidarL2/meshes/unilidarl2base.stl"/>
         </geometry>
       </collision>
     </link>
-    <!-- Reference frame exported by the CAD model for downstream attachments. -->
-    <link name="${prefix}LidarBase">
-      <inertial>
-        <origin xyz="0 0 0" rpy="0 0 0"/>
-        <mass value="1e-9"/>
-        <inertia ixx="0" ixy="0" ixz="0" iyy="0" iyz="0" izz="0"/>
-      </inertial>
-    </link>
-    <joint name="${prefix}LidarBase_frame" type="fixed">
-      <origin xyz="0 0 -0" rpy="0 0 1.5708"/>
-      <parent link="${prefix}unilidarl2base"/>
-      <child link="${prefix}LidarBase"/>
-      <axis xyz="0 0 0"/>
-    </joint>
     <!-- Rotating top cap of the lidar. -->
     <link name="${prefix}unilidarl2top">
       <inertial>
-        <origin xyz="-2.7414e-06 6.66489e-05 -0.0157604" rpy="0 0 0"/>
+        <origin xyz="6.66489e-05 -2.74177e-06 0.0157604" rpy="0 0 0"/>
         <mass value="0.13"/>
-        <inertia ixx="5.78833e-05" ixy="-1.075e-09" ixz="2.975e-09" iyy="3.66094e-05" iyz="9.3857e-08" izz="7.00661e-05"/>
+        <inertia ixx="3.66094e-05" ixy="-1.075e-09" ixz="-9.3857e-08" iyy="5.78833e-05" iyz="-2.975e-09" izz="7.00661e-05"/>
       </inertial>
       <visual>
-        <origin xyz="-0.53025 -1.94934e-06 -0.290634" rpy="-0 0.349066 -0"/>
+        <origin xyz="-1.94934e-06 -0.53025 0.290634" rpy="3.14159 -0.349066 1.5708"/>
         <geometry>
-          <mesh filename="package://kanga_description/meshes/sensors/unilidar_l2/unilidarl2top.stl"/>
+          <mesh filename="package://kanga_description/urdf/sensors/UniLidarL2/meshes/unilidarl2top.stl"/>
         </geometry>
         <material name="unilidarl2top_material">
@@ -68,7 +54,7 @@
       </visual>
       <collision>
-        <origin xyz="-0.53025 -1.94934e-06 -0.290634" rpy="-0 0.349066 -0"/>
+        <origin xyz="-1.94934e-06 -0.53025 0.290634" rpy="3.14159 -0.349066 1.5708"/>
         <geometry>
-          <mesh filename="package://kanga_description/meshes/sensors/unilidar_l2/unilidarl2top.stl"/>
+          <mesh filename="package://kanga_description/urdf/sensors/UniLidarL2/meshes/unilidarl2top.stl"/>
         </geometry>
       </collision>
@@ -76,5 +62,5 @@
     <!-- Spin joint from base to top cap (currently constrained by limits). -->
     <joint name="${prefix}LidarTop" type="revolute">
-      <origin xyz="0 0 0.0226" rpy="3.14159 -0 -3.14159"/>
+      <origin xyz="-0 0 0.0214" rpy="0 -0 0"/>
       <parent link="${prefix}unilidarl2base"/>
       <child link="${prefix}unilidarl2top"/>

Commit message: updated naming schemes

File: kanga_description/onshape_export/UniLidarL2/UniLidarL2.urdf (robot description, URDF)
Before this commit: robot UniLidarL2, 2 links, 1 joints
Links:
- removed link unilidarl2base
- removed link unilidarl2top
- added link unilidarl2_base, mass 0.1; collision mesh filename=package://kanga_description/assets_UniLidarL2/unilidarl2_ba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; visual mesh filename=package://kanga_description/assets_UniLidarL2/unilidarl2_ba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
- added link unilidarl2_top, mass 0.13; collision mesh filename=package://kanga_description/assets_UniLidarL2/unilidarl2_to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; visual mesh filename=package://kanga_description/assets_UniLidarL2/unilidarl2_to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
Joints:
- joint LidarTop: child unilidarl2top -> unilidarl2_top; parent unilidarl2base -> unilidarl2_base

File: kanga_description/onshape_export/autonomous_lidar_payload/autonomous_lidar_payload.urdf (robot description, URDF)
Before this commit: robot autonomous_lidar_payload, 3 links, 2 joints
Links:
- removed link autonomouslidarmount
- link autonomous_lidar_mount: mass 1e-9 -> 0.4; geometry collision mesh filename=package://kanga_description/assets_autonomous_lidar_payload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; visual mesh filename=package://kanga_description/assets_autonomous_lidar_payload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
Joints:
- removed joint autonomous_lidar_mount_frame
- joint unilidarl2_mount_frame: parent autonomouslidarmount -> autonomous_lidar_mount

File: kanga_description/urdf/payloads/autonomous/autonomous_lidar_payload_macro.urdf.xacro (robot description, xacro)
@@ -13,9 +13,9 @@
       <origin xyz="${xyz}" rpy="${rpy}"/>
       <parent link="${parent}"/>
-      <child link="${prefix}autonomouslidarmount"/>
+      <child link="${prefix}autonomous_lidar_mount"/>
       <axis xyz="0 0 0"/>
     </joint>
     <!-- Payload bracket geometry that bolts to rover top mount. -->
-    <link name="${prefix}autonomouslidarmount">
+    <link name="${prefix}autonomous_lidar_mount">
       <inertial>
         <origin xyz="-0.0301856 0.1575 0.184178" rpy="0 0 0"/>
@@ -26,8 +26,8 @@
         <origin xyz="-0.420514 0.1575 -0.1216" rpy="-0 -0 0"/>
         <geometry>
-          <mesh filename="package://kanga_description/meshes/payloads/auto/autonomouslidarmount.stl"/>
+          <mesh filename="package://kanga_description/meshes/payloads/auto/autonomous_lidar_mount.stl"/>
         </geometry>
-        <material name="autonomouslidarmount_material">
-          <color rgba="0.5 0.5 0.5 1"/>
+        <material name="autonomous_lidar_mount_material">
+          <color rgba="0.231373 0.380392 0.705882 1"/>
         </material>
       </visual>
@@ -35,10 +35,10 @@
         <origin xyz="-0.420514 0.1575 -0.1216" rpy="-0 -0 0"/>
         <geometry>
-          <mesh filename="package://kanga_description/meshes/payloads/auto/autonomouslidarmount.stl"/>
+          <mesh filename="package://kanga_description/meshes/payloads/auto/autonomous_lidar_mount.stl"/>
         </geometry>
       </collision>
     </link>
     <!-- Lidar mounting frame exported from CAD for sensor placement. -->
-    <link name="${prefix}UniLidarL2Mount">
+    <link name="${prefix}unilidarl2_mount">
       <inertial>
         <origin xyz="0 0 0" rpy="0 0 0"/>
@@ -47,12 +47,12 @@
       </inertial>
     </link>
-    <joint name="${prefix}UniLidarL2Mount_frame" type="fixed">
+    <joint name="${prefix}unilidarl2_mount_frame" type="fixed">
       <origin xyz="-0.0300581 0.1575 0.355979" rpy="2.79253 -0 1.5708"/>
-      <parent link="${prefix}autonomouslidarmount"/>
-      <child link="${prefix}UniLidarL2Mount"/>
+      <parent link="${prefix}autonomous_lidar_mount"/>
+      <child link="${prefix}unilidarl2_mount"/>
       <axis xyz="0 0 0"/>
     </joint>
     <!-- Attach reusable UniLidarL2 model at the payload's lidar mount frame. -->
-    <xacro:unilidar_l2 parent="${prefix}UniLidarL2Mount" prefix="${prefix}"/>
+    <xacro:unilidar_l2 parent="${prefix}unilidarl2_mount" prefix="${prefix}"/>
   </xacro:macro>
 </robot>

File: kanga_description/urdf/sensors/UniLidarL2/UniLidarL2_macro.urdf.xacro (robot description, xacro)
@@ -11,9 +11,9 @@
       <origin xyz="${xyz}" rpy="${rpy}"/>
       <parent link="${parent}"/>
-      <child link="${prefix}unilidarl2base"/>
+      <child link="${prefix}unilidarl2_base"/>
       <axis xyz="0 0 0"/>
     </joint>
     <!-- Main lidar body. -->
-    <link name="${prefix}unilidarl2base">
+    <link name="${prefix}unilidarl2_base">
       <inertial>
         <origin xyz="6.88756e-05 4.86924e-06 0.00436145" rpy="0 0 0"/>
@@ -24,5 +24,5 @@
         <origin xyz="-1.94934e-06 -0.53025 0.313234" rpy="3.14159 -0.349066 1.5708"/>
         <geometry>
-          <mesh filename="package://kanga_description/urdf/sensors/UniLidarL2/meshes/unilidarl2base.stl"/>
+          <mesh filename="package://kanga_description/urdf/sensors/UniLidarL2/meshes/unilidarl2_base.stl"/>
         </geometry>
         <material name="unilidarl2base_material">
@@ -33,10 +33,10 @@
         <origin xyz="-1.94934e-06 -0.53025 0.313234" rpy="3.14159 -0.349066 1.5708"/>
         <geometry>
-          <mesh filename="package://kanga_description/urdf/sensors/UniLidarL2/meshes/unilidarl2base.stl"/>
+          <mesh filename="package://kanga_description/urdf/sensors/UniLidarL2/meshes/unilidarl2_base.stl"/>
         </geometry>
       </collision>
     </link>
     <!-- Rotating top cap of the lidar. -->
-    <link name="${prefix}unilidarl2top">
+    <link name="${prefix}unilidarl2_top">
       <inertial>
         <origin xyz="6.66489e-05 -2.74177e-06 0.0157604" rpy="0 0 0"/>
@@ -47,5 +47,5 @@
         <origin xyz="-1.94934e-06 -0.53025 0.290634" rpy="3.14159 -0.349066 1.5708"/>
         <geometry>
-          <mesh filename="package://kanga_description/urdf/sensors/UniLidarL2/meshes/unilidarl2top.stl"/>
+          <mesh filename="package://kanga_description/urdf/sensors/UniLidarL2/meshes/unilidarl2_top.stl"/>
         </geometry>
         <material name="unilidarl2top_material">
@@ -56,5 +56,5 @@
         <origin xyz="-1.94934e-06 -0.53025 0.290634" rpy="3.14159 -0.349066 1.5708"/>
         <geometry>
-          <mesh filename="package://kanga_description/urdf/sensors/UniLidarL2/meshes/unilidarl2top.stl"/>
+          <mesh filename="package://kanga_description/urdf/sensors/UniLidarL2/meshes/unilidarl2_top.stl"/>
         </geometry>
       </collision>
@@ -63,6 +63,6 @@
     <joint name="${prefix}LidarTop" type="revolute">
       <origin xyz="-0 0 0.0214" rpy="0 -0 0"/>
-      <parent link="${prefix}unilidarl2base"/>
-      <child link="${prefix}unilidarl2top"/>
+      <parent link="${prefix}unilidarl2_base"/>
+      <child link="${prefix}unilidarl2_top"/>
       <axis xyz="0 0 1"/>
       <limit effort="10" velocity="10" lower="0" upper="0"/>
