Commit message: clean up codebase robot_description

File: kanga_description/urdf/core/kanga_core_macro.urdf.xacro (robot description, xacro)
@@ -2,16 +2,18 @@
 <robot name="kanga_core_macro" xmlns:xacro="http://www.ros.org/wiki/xacro">
   <!-- Reusable rover core model.
-       This macro defines the complete base chassis, payload mount frames, and wheels. -->
-  <xacro:macro name="kanga_core" params="">
+       This macro defines the complete base chassis, payload mount frames, and wheels.
+       Params:
+       - prefix: optional name prefix to avoid link/joint collisions -->
+  <xacro:macro name="kanga_core" params="prefix:=''">
   <!-- Base/root frame for full rover assemblies. -->
-  <link name="base_link"/>
-  <joint name="base_link_to_kangacore" type="fixed">
-    <parent link="base_link"/>
-    <child link="kanga_core"/>
+  <link name="${prefix}base_link"/>
+  <joint name="${prefix}base_link_to_kanga_core" type="fixed">
+    <parent link="${prefix}base_link"/>
+    <child link="${prefix}kanga_core"/>
     <!-- <origin xyz="0.55486398 0.44572500 0.39697" rpy="0 0 1.5708"/> -->
     <origin xyz="0.0 0.0 0.39697" rpy="0 0 0"/>
   </joint>
   <!-- Main chassis body geometry + inertial properties. -->
-  <link name="kanga_core">
+  <link name="${prefix}kanga_core">
     <inertial>
       <origin xyz="-0.0394422 -0.0149606 -0.0298892" rpy="0 0 0"/>
@@ -37,5 +39,5 @@
   </link>
   <!-- Top payload interface frame used by payload assemblies. -->
-  <link name="top_payload_mount">
+  <link name="${prefix}top_payload_mount">
     <inertial>
       <origin xyz="0 0 0" rpy="0 0 0"/>
@@ -44,12 +46,12 @@
     </inertial>
   </link>
-  <joint name="top_payload_mount_frame" type="fixed">
+  <joint name="${prefix}top_payload_mount_frame" type="fixed">
     <origin xyz="0.379844 -0.1575 0.1216" rpy="0 -0 0"/>
-    <parent link="kanga_core"/>
-    <child link="top_payload_mount"/>
+    <parent link="${prefix}kanga_core"/>
+    <child link="${prefix}top_payload_mount"/>
     <axis xyz="0 0 0"/>
   </joint>
   <!-- Front payload interface frame used by payload assemblies. -->
-  <link name="front_payload_mount">
+  <link name="${prefix}front_payload_mount">
     <inertial>
       <origin xyz="0 0 0" rpy="0 0 0"/>
@@ -58,13 +60,13 @@
     </inertial>
   </link>
-  <joint name="front_payload_mount_frame" type="fixed">
+  <joint name="${prefix}front_payload_mount_frame" type="fixed">
     <origin xyz="0.158499 -0 0.0116" rpy="0 -0 0"/>
-    <parent link="kanga_core"/>
-    <child link="front_payload_mount"/>
+    <parent link="${prefix}kanga_core"/>
+    <child link="${prefix}front_payload_mount"/>
     <axis xyz="0 0 0"/>
   </joint>
   <!-- Drive wheel links and joints. -->
-  <!-- Link wheel_FL -->
-  <link name="wheel_FL">
+  <!-- Link wheel_fl -->
+  <link name="${prefix}wheel_fl">
     <inertial>
       <origin xyz="8.20141e-07 4.19108e-07 0.0294338" rpy="0 0 0"/>
@@ -89,14 +91,14 @@
     </collision>
   </link>
-  <!-- Joint from kanga_core to wheel_FL -->
-  <joint name="wheel1" type="continuous">
+  <!-- Joint from kanga_core to wheel_fl -->
+  <joint name="${prefix}wheel_fl_joint" type="continuous">
     <origin xyz="0.428413 0.395775 -0.271989" rpy="1.5708 0 0"/>
-    <parent link="kanga_core"/>
-    <child link="wheel_FL"/>
+    <parent link="${prefix}kanga_core"/>
+    <child link="${prefix}wheel_fl"/>
     <axis xyz="0 0 1"/>
     <limit effort="40" velocity="4.61"/>
   </joint>
-  <!-- Link wheel_BL -->
-  <link name="wheel_BL">
+  <!-- Link wheel_bl -->
+  <link name="${prefix}wheel_bl">
     <inertial>
       <origin xyz="1.69548e-06 -4.25166e-07 0.0294802" rpy="0 0 0"/>
@@ -121,14 +123,14 @@
     </collision>
   </link>
-  <!-- Joint from kanga_core to wheel_BL -->
-  <joint name="wheel2" type="continuous">
+  <!-- Joint from kanga_core to wheel_bl -->
+  <joint name="${prefix}wheel_bl_joint" type="continuous">
     <origin xyz="-0.430143 0.395775 -0.272479" rpy="1.5708 0 -0"/>
-    <parent link="kanga_core"/>
-    <child link="wheel_BL"/>
+    <parent link="${prefix}kanga_core"/>
+    <child link="${prefix}wheel_bl"/>
     <axis xyz="0 0 1"/>
     <limit effort="40" velocity="4.61"/>
   </joint>
-  <!-- Link wheel_BR -->
-  <link name="wheel_BR">
+  <!-- Link wheel_br -->
+  <link name="${prefix}wheel_br">
     <inertial>
       <origin xyz="8.20141e-07 4.19108e-07 0.0294338" rpy="0 0 0"/>
@@ -153,14 +155,14 @@
     </collision>
   </link>
-  <!-- Joint from kanga_core to wheel_BR -->
-  <joint name="wheel3" type="continuous">
+  <!-- Joint from kanga_core to wheel_br -->
+  <joint name="${prefix}wheel_br_joint" type="continuous">
     <origin xyz="-0.430143 -0.395725 -0.272479" rpy="1.5708 0 -3.14159"/>
-    <parent link="kanga_core"/>
-    <child link="wheel_BR"/>
+    <parent link="${prefix}kanga_core"/>
+    <child link="${prefix}wheel_br"/>
     <axis xyz="0 0 1"/>
     <limit effort="40" velocity="4.61"/>
   </joint>
-  <!-- Link wheel_FR -->
-  <link name="wheel_FR">
+  <!-- Link wheel_fr -->
+  <link name="${prefix}wheel_fr">
     <inertial>
       <origin xyz="1.69548e-06 -4.25166e-07 0.0294802" rpy="0 0 0"/>
@@ -185,9 +187,9 @@
     </collision>
   </link>
-  <!-- Joint from kanga_core to wheel_FR -->
-  <joint name="wheel4" type="continuous">
+  <!-- Joint from kanga_core to wheel_fr -->
+  <joint name="${prefix}wheel_fr_joint" type="continuous">
     <origin xyz="0.428413 -0.395725 -0.271989" rpy="1.5708 -0 -3.14159"/>
-    <parent link="kanga_core"/>
-    <child link="wheel_FR"/>
+    <parent link="${prefix}kanga_core"/>
+    <child link="${prefix}wheel_fr"/>
     <axis xyz="0 0 1"/>
     <limit effort="40" velocity="4.61"/>

File: kanga_description/urdf/payloads/autonomous/autonomous_lidar_payload_macro.urdf.xacro (robot description, xacro)
@@ -10,5 +10,5 @@
   <xacro:macro name="autonomous_lidar_payload" params="parent xyz:='0 0 0' rpy:='0 0 0' prefix:=''">
     <!-- Mount payload body to caller-provided parent link. -->
-    <joint name="${prefix}autonomous_payload_mount_joint" type="fixed">
+    <joint name="${prefix}autonomous_lidar_payload_mount_joint" type="fixed">
       <origin xyz="${xyz}" rpy="${rpy}"/>
       <parent link="${parent}"/>
@@ -54,5 +54,5 @@
     </joint>
     <!-- Attach reusable UniLidarL2 model at the payload's lidar mount frame. -->
-    <xacro:unilidar_l2 parent="${prefix}unilidarl2_mount" prefix="${prefix}"/>
+    <xacro:unilidarl2 parent="${prefix}unilidarl2_mount" prefix="${prefix}"/>
   </xacro:macro>
 </robot>

File: kanga_description/urdf/sensors/UniLidarL2/UniLidarL2_descr.urdf.xacro (robot description, xacro)
@@ -1,4 +1,4 @@
 <?xml version="1.0" ?>
-<robot name="UniLidarL2" xmlns:xacro="http://www.ros.org/wiki/xacro">
+<robot name="unilidarl2" xmlns:xacro="http://www.ros.org/wiki/xacro">
   <!-- Wrapper file:
        Include the reusable lidar macro and instantiate it as a standalone model. -->
@@ -7,4 +7,4 @@
   <link name="base_link"/>
   <!-- Instantiate the reusable macro and attach it to this root. -->
-  <xacro:unilidar_l2 parent="base_link"/>
+  <xacro:unilidarl2 parent="base_link"/>
 </robot>

File: kanga_description/urdf/sensors/UniLidarL2/UniLidarL2_macro.urdf.xacro (robot description, xacro)
@@ -1,4 +1,4 @@
 <?xml version="1.0" ?>
-<robot name="UniLidarL2_macro" xmlns:xacro="http://www.ros.org/wiki/xacro">
+<robot name="unilidarl2_macro" xmlns:xacro="http://www.ros.org/wiki/xacro">
   <!-- Reusable lidar component.
        Params:
@@ -6,7 +6,7 @@
        - xyz/rpy: pose of the lidar relative to parent
        - prefix: optional name prefix to avoid link/joint collisions -->
-  <xacro:macro name="unilidar_l2" params="parent xyz:='0 0 0' rpy:='0 0 0' prefix:=''">
+  <xacro:macro name="unilidarl2" params="parent xyz:='0 0 0' rpy:='0 0 0' prefix:=''">
     <!-- Mount joint from caller-provided parent to lidar base. -->
-    <joint name="${prefix}UniLidarL2_mount_joint" type="fixed">
+    <joint name="${prefix}unilidarl2_mount_joint" type="fixed">
       <origin xyz="${xyz}" rpy="${rpy}"/>
       <parent link="${parent}"/>
@@ -26,5 +26,5 @@
           <mesh filename="package://kanga_description/urdf/sensors/UniLidarL2/meshes/unilidarl2_base.stl"/>
         </geometry>
-        <material name="unilidarl2base_material">
+        <material name="unilidarl2_base_material">
           <color rgba="0.301961 0.301961 0.301961 1"/>
         </material>
@@ -49,5 +49,5 @@
           <mesh filename="package://kanga_description/urdf/sensors/UniLidarL2/meshes/unilidarl2_top.stl"/>
         </geometry>
-        <material name="unilidarl2top_material">
+        <material name="unilidarl2_top_material">
           <color rgba="0.215686 0.215686 0.215686 1"/>
         </material>
@@ -61,5 +61,5 @@
     </link>
     <!-- Spin joint from base to top cap (currently constrained by limits). -->
-    <joint name="${prefix}LidarTop" type="revolute">
+    <joint name="${prefix}unilidarl2_top_joint" type="revolute">
       <origin xyz="-0 0 0.0214" rpy="0 -0 0"/>
       <parent link="${prefix}unilidarl2_base"/>
