Commit message: stuff

File: kanga_description/urdf/core/kanga_core_simple_macro.urdf.xacro (robot description, xacro)
@@ -31,8 +31,26 @@
       </material>
     </visual>
-    <collision>
+    <!-- <collision>
       <origin xyz="-0.0406693 -0 0" rpy="0 -0 1.5708"/>
       <geometry>
         <mesh filename="package://kanga_description/meshes/core/kangacore.stl"/>
+      </geometry>
+    </collision> -->
+    <collision>
+      <origin xyz="0.0 -0 0.5" rpy="0 -0 1.5708"/>
+      <geometry>
+        <box size="0.45 0.9 1.2"/>
+      </geometry>
+    </collision>
+    <collision>
+      <origin xyz="0 0.32 -0.2" rpy="0 -0 1.5708"/>
+      <geometry>
+        <box size="0.3 1.3 0.6"/>
+      </geometry>
+    </collision>
+    <collision>
+      <origin xyz="0 -0.32 -0.2" rpy="0 -0 1.5708"/>
+      <geometry>
+        <box size="0.3 1.3 0.6"/>
       </geometry>
     </collision>
@@ -85,7 +103,7 @@
     </visual>
     <collision>
-      <origin xyz="0 0 -0.05" rpy="-1.5708 -0 0"/>
-      <geometry>
-        <mesh filename="package://kanga_description/meshes/core/wheelb.stl"/>
+      <origin xyz="0 0 0.08" rpy="0 0 0"/>
+      <geometry>
+        <cylinder radius="0.126" length="0.3"/>
       </geometry>
     </collision>
@@ -117,7 +135,7 @@
     </visual>
     <collision>
-      <origin xyz="0 0 -0.05" rpy="-1.5708 0 0"/>
-      <geometry>
-        <mesh filename="package://kanga_description/meshes/core/wheel_a.stl"/>
+      <origin xyz="0 0 0.08" rpy="0 0 0"/>
+      <geometry>
+        <cylinder radius="0.126" length="0.3"/>
       </geometry>
     </collision>
@@ -149,7 +167,7 @@
     </visual>
     <collision>
-      <origin xyz="0 0 -0.05" rpy="-1.5708 0 0"/>
-      <geometry>
-        <mesh filename="package://kanga_description/meshes/core/wheelb.stl"/>
+      <origin xyz="0 0 0.08" rpy="0 0 0"/>
+      <geometry>
+        <cylinder radius="0.126" length="0.3"/>
       </geometry>
     </collision>
@@ -181,7 +199,7 @@
     </visual>
     <collision>
-      <origin xyz="0 0 -0.05" rpy="-1.5708 -0 0"/>
-      <geometry>
-        <mesh filename="package://kanga_description/meshes/core/wheel_a.stl"/>
+      <origin xyz="0 0 0.08" rpy="0 0 0"/>
+      <geometry>
+        <cylinder radius="0.126" length="0.3"/>
       </geometry>
     </collision>
