Commit message: Added a simple and a non simple variant of the core where suspension is split

File: kanga_description/onshape_export/kanga_core/kanga_core.urdf (robot description, URDF)
Before this commit: robot kanga_core, 7 links, 6 joints
Links:
- removed link base_link
- added link antenna, mass 8.4; collision mesh filename=package://kanga_description/assets_kanga_core/antenna.stl; collision mesh filename=package://kanga_description/assets_kanga_core/core.stl
- added link diff_bar, mass 0.4; collision mesh filename=package://kanga_description/assets_kanga_core/diff_bar.stl; visual mesh filename=package://kanga_description/assets_kanga_core/diff_bar.stl
- added link left_suspension, mass 9; collision mesh filename=package://kanga_description/assets_kanga_core/left_suspensi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; visual mesh filename=package://kanga_description/assets_kanga_core/left_suspensi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
- added link right_suspension, mass 9; collision mesh filename=package://kanga_description/assets_kanga_core/right_suspens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; visual mesh filename=package://kanga_description/assets_kanga_core/right_suspens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
- link wheel_a: geometry collision mesh filename=package://kanga_description/assets_kanga_core/wheel_a.stl; visual mesh filename=package://kanga_description/assets_kanga_core/wheel_a.stl
- link wheel_a_2: geometry collision mesh filename=package://kanga_description/assets_kanga_core/wheel_a.stl; visual mesh filename=package://kanga_description/assets_kanga_core/wheel_a.stl
- link wheelb: geometry collision mesh filename=package://kanga_description/assets_kanga_core/wheelb.stl; visual mesh filename=package://kanga_description/assets_kanga_core/wheelb.stl
- link wheelb_2: geometry collision mesh filename=package://kanga_description/assets_kanga_core/wheelb.stl; visual mesh filename=package://kanga_description/assets_kanga_core/wheelb.stl
Joints:
- removed joint wheel1
- removed joint wheel2
- removed joint wheel3
- removed joint wheel4
- added joint diff_bar: type revolute, parent antenna, child diff_bar, origin xyz=-0.301156 0 0.0766 rpy=1.5708 0 1.5708, axis 0 0 1, limit lower=0 upper=0 effort=0 velocity=0
- added joint left_suspension: type revolute, parent antenna, child left_suspension, origin xyz=0.148499 0.1911 0.0616 rpy=1.5708 0 0, axis 0 0 1, limit lower=0 upper=0 effort=0 velocity=0
- added joint right_suspension: type revolute, parent antenna, child right_suspension, origin xyz=0.148499 -0.1911 0.0616 rpy=1.5708 -0 -3.14159, axis 0 0 1, limit lower=0 upper=0 effort=0 velocity=0
- added joint wheel_bl: type continuous, parent left_suspension, child wheel_a, origin xyz=-0.578642 -0.334079 -0.204675 rpy=-0 -0 0, axis 0 0 1, limit lower=0 upper=0 effort=0 velocity=0
- added joint wheel_br: type continuous, parent right_suspension, child wheelb_2, origin xyz=0.578642 -0.334079 -0.204625 rpy=-0 -0 0, axis 0 0 1, limit effort=0 velocity=0
- added joint wheel_fl: type continuous, parent left_suspension, child wheelb, origin xyz=0.279914 -0.333589 -0.204675 rpy=0 -0 -0, axis 0 0 1, limit effort=0 velocity=0
- added joint wheel_fr: type continuous, parent right_suspension, child wheel_a_2, origin xyz=-0.279914 -0.333589 -0.204625 rpy=0 -0 -0, axis 0 0 1, limit effort=0 velocity=0
- joint front_payload_mount_frame: origin xyz=0.158499 -0 0.0116 rpy=0 -0 0 -> xyz=0.158499 -0 0.0116 rpy=0 0 0; parent base_link -> antenna
- joint top_payload_mount_frame: origin xyz=0.379844 -0.1575 0.1216 rpy=0 -0 0 -> xyz=0.379844 -0.1575 0.1216 rpy=-0 0 0; parent base_link -> antenna

File: kanga_description/urdf/core/kanga_core_macro.urdf.xacro (robot description, xacro)
@@ -1,198 +1,282 @@
 <?xml version="1.0" ?>
 <robot name="kanga_core_macro" xmlns:xacro="http://www.ros.org/wiki/xacro">
-  <!-- Reusable rover core model.
-       This macro defines the complete base chassis, payload mount frames, and wheels.
+  <!-- Reusable rover core model with suspension.
        Params:
        - prefix: optional name prefix to avoid link/joint collisions -->
   <xacro:macro name="kanga_core" params="prefix:=''">
-  <!-- Base/root frame for full rover assemblies. -->
-  <link name="${prefix}base_link"/>
-  <joint name="${prefix}base_link_to_kanga_core" type="fixed">
-    <parent link="${prefix}base_link"/>
-    <child link="${prefix}kanga_core"/>
-    <!-- <origin xyz="0.55486398 0.44572500 0.39697" rpy="0 0 1.5708"/> -->
-    <origin xyz="0.0 0.0 0.39697" rpy="0 0 0"/>
-  </joint>
-  <!-- Main chassis body geometry + inertial properties. -->
-  <link name="${prefix}kanga_core">
-    <inertial>
-      <origin xyz="-0.0394422 -0.0149606 -0.0298892" rpy="0 0 0"/>
-      <mass value="28"/>
-      <inertia ixx="3.05326" ixy="-0.0953345" ixz="0.403632" iyy="4.37258" iyz="0.249778" izz="3.81615"/>
-    </inertial>
-    <!-- Part kangacore -->
-    <visual>
-      <origin xyz="-0.0406693 -0 0" rpy="0 -0 1.5708"/>
-      <geometry>
-        <mesh filename="package://kanga_description/meshes/core/kangacore.stl"/>
-      </geometry>
-      <material name="kangacore_material">
-        <color rgba="0.917647 0.917647 0.917647 1"/>
-      </material>
-    </visual>
-    <collision>
-      <origin xyz="-0.0406693 -0 0" rpy="0 -0 1.5708"/>
-      <geometry>
-        <mesh filename="package://kanga_description/meshes/core/kangacore.stl"/>
-      </geometry>
-    </collision>
-  </link>
-  <!-- Top payload interface frame used by payload assemblies. -->
-  <link name="${prefix}top_payload_mount">
-    <inertial>
-      <origin xyz="0 0 0" rpy="0 0 0"/>
-      <mass value="1e-9"/>
-      <inertia ixx="0" ixy="0" ixz="0" iyy="0" iyz="0" izz="0"/>
-    </inertial>
-  </link>
-  <joint name="${prefix}top_payload_mount_frame" type="fixed">
-    <origin xyz="0.379844 -0.1575 0.1216" rpy="0 -0 0"/>
-    <parent link="${prefix}kanga_core"/>
-    <child link="${prefix}top_payload_mount"/>
-    <axis xyz="0 0 0"/>
-  </joint>
-  <!-- Front payload interface frame used by payload assemblies. -->
-  <link name="${prefix}front_payload_mount">
-    <inertial>
-      <origin xyz="0 0 0" rpy="0 0 0"/>
-      <mass value="1e-9"/>
-      <inertia ixx="0" ixy="0" ixz="0" iyy="0" iyz="0" izz="0"/>
-    </inertial>
-  </link>
-  <joint name="${prefix}front_payload_mount_frame" type="fixed">
-    <origin xyz="0.158499 -0 0.0116" rpy="0 -0 0"/>
-    <parent link="${prefix}kanga_core"/>
-    <child link="${prefix}front_payload_mount"/>
-    <axis xyz="0 0 0"/>
-  </joint>
-  <!-- Drive wheel links and joints. -->
-  <!-- Link wheel_fl -->
-  <link name="${prefix}wheel_fl">
-    <inertial>
-      <origin xyz="8.20141e-07 4.19108e-07 0.0294338" rpy="0 0 0"/>
-      <mass value="0.7"/>
-      <inertia ixx="0.00536519" ixy="2.6367e-08" ixz="3.55462e-07" iyy="0.00536521" iyz="7.378e-09" izz="0.00759451"/>
-    </inertial>
-    <!-- Part wheelb -->
-    <visual>
-      <origin xyz="0 0 -0.05" rpy="-1.5708 -0 0"/>
-      <geometry>
-        <mesh filename="package://kanga_description/meshes/core/wheelb.stl"/>
-      </geometry>
-      <material name="wheelb_material">
-        <color rgba="0.929412 0.0392157 0 1"/>
-      </material>
-    </visual>
-    <collision>
-      <origin xyz="0 0 -0.05" rpy="-1.5708 -0 0"/>
-      <geometry>
-        <mesh filename="package://kanga_description/meshes/core/wheelb.stl"/>
-      </geometry>
-    </collision>
-  </link>
-  <!-- Joint from kanga_core to wheel_fl -->
-  <joint name="${prefix}wheel_fl_joint" type="continuous">
-    <origin xyz="0.428413 0.395775 -0.271989" rpy="1.5708 0 0"/>
-    <parent link="${prefix}kanga_core"/>
-    <child link="${prefix}wheel_fl"/>
-    <axis xyz="0 0 1"/>
-    <limit effort="40" velocity="4.61"/>
-  </joint>
-  <!-- Link wheel_bl -->
-  <link name="${prefix}wheel_bl">
-    <inertial>
-      <origin xyz="1.69548e-06 -4.25166e-07 0.0294802" rpy="0 0 0"/>
-      <mass value="0.7"/>
-      <inertia ixx="0.0053658" ixy="2.7862e-08" ixz="3.79976e-07" iyy="0.00536582" iyz="-5.263e-09" izz="0.00759416"/>
-    </inertial>
-    <!-- Part wheel_a -->
-    <visual>
-      <origin xyz="0 0 -0.05" rpy="-1.5708 0 0"/>
-      <geometry>
-        <mesh filename="package://kanga_description/meshes/core/wheel_a.stl"/>
-      </geometry>
-      <material name="wheel_a_material">
-        <color rgba="0.929412 0.0392157 0 1"/>
-      </material>
-    </visual>
-    <collision>
-      <origin xyz="0 0 -0.05" rpy="-1.5708 0 0"/>
-      <geometry>
-        <mesh filename="package://kanga_description/meshes/core/wheel_a.stl"/>
-      </geometry>
-    </collision>
-  </link>
-  <!-- Joint from kanga_core to wheel_bl -->
-  <joint name="${prefix}wheel_bl_joint" type="continuous">
-    <origin xyz="-0.430143 0.395775 -0.272479" rpy="1.5708 0 -0"/>
-    <parent link="${prefix}kanga_core"/>
-    <child link="${prefix}wheel_bl"/>
-    <axis xyz="0 0 1"/>
-    <limit effort="40" velocity="4.61"/>
-  </joint>
-  <!-- Link wheel_br -->
-  <link name="${prefix}wheel_br">
-    <inertial>
-      <origin xyz="8.20141e-07 4.19108e-07 0.0294338" rpy="0 0 0"/>
-      <mass value="0.7"/>
-      <inertia ixx="0.00536519" ixy="2.6367e-08" ixz="3.55462e-07" iyy="0.00536521" iyz="7.378e-09" izz="0.00759451"/>
-    </inertial>
-    <!-- Part wheelb_2 -->
-    <visual>
-      <origin xyz="0 0 -0.05" rpy="-1.5708 0 0"/>
-      <geometry>
-        <mesh filename="package://kanga_description/meshes/core/wheelb.stl"/>
-      </geometry>
-      <material name="wheelb_2_material">
-        <color rgba="0.929412 0.0392157 0 1"/>
-      </material>
-    </visual>
-    <collision>
-      <origin xyz="0 0 -0.05" rpy="-1.5708 0 0"/>
-      <geometry>
-        <mesh filename="package://kanga_description/meshes/core/wheelb.stl"/>
-      </geometry>
-    </collision>
-  </link>
-  <!-- Joint from kanga_core to wheel_br -->
-  <joint name="${prefix}wheel_br_joint" type="continuous">
-    <origin xyz="-0.430143 -0.395725 -0.272479" rpy="1.5708 0 -3.14159"/>
-    <parent link="${prefix}kanga_core"/>
-    <child link="${prefix}wheel_br"/>
-    <axis xyz="0 0 1"/>
-    <limit effort="40" velocity="4.61"/>
-  </joint>
-  <!-- Link wheel_fr -->
-  <link name="${prefix}wheel_fr">
-    <inertial>
-      <origin xyz="1.69548e-06 -4.25166e-07 0.0294802" rpy="0 0 0"/>
-      <mass value="0.7"/>
-      <inertia ixx="0.0053658" ixy="2.7862e-08" ixz="3.79976e-07" iyy="0.00536582" iyz="-5.263e-09" izz="0.00759416"/>
-    </inertial>
-    <!-- Part wheel_a_2 -->
-    <visual>
-      <origin xyz="0 0 -0.05" rpy="-1.5708 -0 0"/>
-      <geometry>
-        <mesh filename="package://kanga_description/meshes/core/wheel_a.stl"/>
-      </geometry>
-      <material name="wheel_a_2_material">
-        <color rgba="0.929412 0.0392157 0 1"/>
-      </material>
-    </visual>
-    <collision>
-      <origin xyz="0 0 -0.05" rpy="-1.5708 -0 0"/>
-      <geometry>
-        <mesh filename="package://kanga_description/meshes/core/wheel_a.stl"/>
-      </geometry>
-    </collision>
-  </link>
-  <!-- Joint from kanga_core to wheel_fr -->
-  <joint name="${prefix}wheel_fr_joint" type="continuous">
-    <origin xyz="0.428413 -0.395725 -0.271989" rpy="1.5708 -0 -3.14159"/>
-    <parent link="${prefix}kanga_core"/>
-    <child link="${prefix}wheel_fr"/>
-    <axis xyz="0 0 1"/>
-    <limit effort="40" velocity="4.61"/>
-  </joint>
+    <!-- Base/root frame for full rover assemblies. -->
+    <link name="${prefix}base_link"/>
+    <joint name="${prefix}base_link_to_kanga_core" type="fixed">
+      <parent link="${prefix}base_link"/>
+      <child link="${prefix}kanga_core"/>
+      <origin xyz="0.0 0.0 0.39697" rpy="0 0 0"/>
+    </joint>
+    <!-- Main chassis body (core + antenna geometry). -->
+    <link name="${prefix}kanga_core">
+      <inertial>
+        <origin xyz="-0.0805841 -0.0158605 0.124198" rpy="0 0 0"/>
+        <mass value="8.4"/>
+        <inertia ixx="0.334932" ixy="-0.0282303" ixz="0.0776441" iyy="0.445283" iyz="0.0534754" izz="0.396654"/>
+      </inertial>
+      <visual>
+        <origin xyz="-0.0406693 -0 0" rpy="0 0 1.5708"/>
+        <geometry>
+          <mesh filename="package://kanga_description/meshes/core/kanga_core/core.stl"/>
+        </geometry>
+        <material name="core_material">
+          <color rgba="0.701961 0.701961 0.701961 1"/>
+        </material>
+      </visual>
+      <collision>
+        <origin xyz="-0.0406693 -0 0" rpy="0 0 1.5708"/>
+        <geometry>
+          <mesh filename="package://kanga_description/meshes/core/kanga_core/core.stl"/>
+        </geometry>
+      </collision>
+      <visual>
+        <origin xyz="-0.0406693 -0 0" rpy="0 -0 1.5708"/>
+        <geometry>
+          <mesh filename="package://kanga_description/meshes/core/kanga_core/antenna.stl"/>
+        </geometry>
+        <material name="antenna_material">
+          <color rgba="0.901961 0.901961 0.901961 1"/>
+        </material>
+      </visual>
+      <collision>
+        <origin xyz="-0.0406693 -0 0" rpy="0 -0 1.5708"/>
+        <geometry>
+          <mesh filename="package://kanga_description/meshes/core/kanga_core/antenna.stl"/>
+        </geometry>
+      </collision>
+    </link>
+    <link name="${prefix}top_payload_mount">
+      <inertial>
+        <origin xyz="0 0 0" rpy="0 0 0"/>
+        <mass value="1e-9"/>
+        <inertia ixx="0" ixy="0" ixz="0" iyy="0" iyz="0" izz="0"/>
+      </inertial>
+    </link>
+    <joint name="${prefix}top_payload_mount_frame" type="fixed">
+      <origin xyz="0.379844 -0.1575 0.1216" rpy="-0 0 0"/>
+      <parent link="${prefix}kanga_core"/>
+      <child link="${prefix}top_payload_mount"/>
+      <axis xyz="0 0 0"/>
+    </joint>
+    <link name="${prefix}front_payload_mount">
+      <inertial>
+        <origin xyz="0 0 0" rpy="0 0 0"/>
+        <mass value="1e-9"/>
+        <inertia ixx="0" ixy="0" ixz="0" iyy="0" iyz="0" izz="0"/>
+      </inertial>
+    </link>
+    <joint name="${prefix}front_payload_mount_frame" type="fixed">
+      <origin xyz="0.158499 -0 0.0116" rpy="0 0 0"/>
+      <parent link="${prefix}kanga_core"/>
+      <child link="${prefix}front_payload_mount"/>
+      <axis xyz="0 0 0"/>
+    </joint>
+    <link name="${prefix}left_suspension">
+      <inertial>
+        <origin xyz="-0.132214 -0.267383 -0.0630324" rpy="0 0 0"/>
+        <mass value="9"/>
+        <inertia ixx="0.143475" ixy="-0.0477444" ixz="-0.00738433" iyy="1.29898" iyz="-0.0240894" izz="1.38116"/>
+      </inertial>
+      <visual>
+        <origin xyz="-0.189168 -0.0616 0.1911" rpy="-1.5708 1.5708 0"/>
+        <geometry>
+          <mesh filename="package://kanga_description/meshes/core/kanga_core/left_suspension.stl"/>
+        </geometry>
+        <material name="left_suspension_material">
+          <color rgba="0.701961 0.701961 0.701961 1"/>
+        </material>
+      </visual>
+      <collision>
+        <origin xyz="-0.189168 -0.0616 0.1911" rpy="-1.5708 1.5708 0"/>
+        <geometry>
+          <mesh filename="package://kanga_description/meshes/core/kanga_core/left_suspension.stl"/>
+        </geometry>
+      </collision>
+    </link>
+    <link name="${prefix}wheel_fl">
+      <inertial>
+        <origin xyz="8.20141e-07 4.19108e-07 0.0294338" rpy="0 0 0"/>
+        <mass value="0.7"/>
+        <inertia ixx="0.00536519" ixy="2.6367e-08" ixz="3.55462e-07" iyy="0.00536521" iyz="7.378e-09" izz="0.00759451"/>
+      </inertial>
+      <visual>
+        <origin xyz="0 -0 -0.05" rpy="-1.5708 0 0"/>
+        <geometry>
+          <mesh filename="package://kanga_description/meshes/core/kanga_core/wheelb.stl"/>
+        </geometry>
+        <material name="wheelb_material">
+          <color rgba="0.929412 0.0392157 0 1"/>
+        </material>
+      </visual>
+      <collision>
+        <origin xyz="0 -0 -0.05" rpy="-1.5708 0 0"/>
+        <geometry>
+          <mesh filename="package://kanga_description/meshes/core/kanga_core/wheelb.stl"/>
+        </geometry>
+      </collision>
+    </link>
+    <joint name="${prefix}wheel_fl_joint" type="continuous">
+      <origin xyz="0.279914 -0.333589 -0.204675" rpy="0 0 0"/>
+      <parent link="${prefix}left_suspension"/>
+      <child link="${prefix}wheel_fl"/>
+      <axis xyz="0 0 1"/>
+      <limit effort="0" velocity="0"/>
+    </joint>
+    <link name="${prefix}wheel_bl">
+      <inertial>
+        <origin xyz="1.69548e-06 -4.25166e-07 0.0294802" rpy="0 0 0"/>
+        <mass value="0.7"/>
+        <inertia ixx="0.0053658" ixy="2.7862e-08" ixz="3.79976e-07" iyy="0.00536582" iyz="-5.263e-09" izz="0.00759416"/>
+      </inertial>
+      <visual>
+        <origin xyz="0 0 -0.05" rpy="-1.5708 -0 0"/>
+        <geometry>
+          <mesh filename="package://kanga_description/meshes/core/kanga_core/wheel_a.stl"/>
+        </geometry>
+        <material name="wheel_a_material">
+          <color rgba="0.929412 0.0392157 0 1"/>
+        </material>
+      </visual>
+      <collision>
+        <origin xyz="0 0 -0.05" rpy="-1.5708 -0 0"/>
+        <geometry>
+          <mesh filename="package://kanga_description/meshes/core/kanga_core/wheel_a.stl"/>
+        </geometry>
+      </collision>
+    </link>
+    <joint name="${prefix}wheel_bl_joint" type="continuous">
+      <origin xyz="-0.578642 -0.334079 -0.204675" rpy="0 0 0"/>
+      <parent link="${prefix}left_suspension"/>
+      <child link="${prefix}wheel_bl"/>
+      <axis xyz="0 0 1"/>
+      <limit effort="0" velocity="0" lower="0" upper="0"/>
+    </joint>
+    <joint name="${prefix}left_suspension_joint" type="revolute">
+      <origin xyz="0.148499 0.1911 0.0616" rpy="1.5708 0 0"/>
+      <parent link="${prefix}kanga_core"/>
+      <child link="${prefix}left_suspension"/>
+      <axis xyz="0 0 1"/>
+      <limit effort="0" velocity="0" lower="0" upper="0"/>
+    </joint>
+    <link name="${prefix}right_suspension">
+      <inertial>
+        <origin xyz="0.134107 -0.26778 -0.0627896" rpy="0 0 0"/>
+        <mass value="9"/>
+        <inertia ixx="0.143252" ixy="0.0492184" ixz="0.00651663" iyy="1.30123" iyz="-0.0237955" izz="1.38328"/>
+      </inertial>
+      <visual>
+        <origin xyz="0.189168 -0.0616 0.1911" rpy="-1.5708 -1.5708 0"/>
+        <geometry>
+          <mesh filename="package://kanga_description/meshes/core/kanga_core/right_suspension.stl"/>
+        </geometry>
+        <material name="right_suspension_material">
+          <color rgba="0.701961 0.701961 0.701961 1"/>
+        </material>
+      </visual>
+      <collision>
+        <origin xyz="0.189168 -0.0616 0.1911" rpy="-1.5708 -1.5708 0"/>
+        <geometry>
+          <mesh filename="package://kanga_description/meshes/core/kanga_core/right_suspension.stl"/>
+        </geometry>
+      </collision>
+    </link>
+    <link name="${prefix}wheel_fr">
+      <inertial>
+        <origin xyz="1.69548e-06 -4.25166e-07 0.0294802" rpy="0 0 0"/>
+        <mass value="0.7"/>
+        <inertia ixx="0.0053658" ixy="2.7862e-08" ixz="3.79976e-07" iyy="0.00536582" iyz="-5.263e-09" izz="0.00759416"/>
+      </inertial>
+      <visual>
+        <origin xyz="0 0 -0.05" rpy="-1.5708 -0 0"/>
+        <geometry>
+          <mesh filename="package://kanga_description/meshes/core/kanga_core/wheel_a.stl"/>
+        </geometry>
+        <material name="wheel_a_2_material">
+          <color rgba="0.929412 0.0392157 0 1"/>
+        </material>
+      </visual>
+      <collision>
+        <origin xyz="0 0 -0.05" rpy="-1.5708 -0 0"/>
+        <geometry>
+          <mesh filename="package://kanga_description/meshes/core/kanga_core/wheel_a.stl"/>
+        </geometry>
+      </collision>
+    </link>
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