Commit message: modified kanga_description files

File: kanga_description/urdf/payloads/arm/arm_payload_macro.urdf.xacro (robot description, xacro)
@@ -199,6 +199,6 @@
       <parent link="${prefix}link2"/>
       <child link="${prefix}link3"/>
-      <axis xyz="0 0 1"/>
-      <limit effort="10" velocity="10" lower="-1.309" upper="2.26893"/>
+      <axis xyz="0 0 -1"/>
+      <limit effort="10" velocity="10" lower="-2.26893" upper="1.309"/>
     </joint>
     <joint name="${prefix}arm_j2" type="revolute">
@@ -213,5 +213,5 @@
       <parent link="${prefix}baserotation"/>
       <child link="${prefix}link1"/>
-      <axis xyz="0 0 1"/>
+      <axis xyz="0 0 -1"/>
       <limit effort="10" velocity="10" lower="-1.5708" upper="1.5708"/>
     </joint>
