Commit message: remote control joint by joint control of arm from base station

File: kanga_arm/kanga_arm_description/urdf/kanga_arm.urdf (robot description, URDF)
Before this commit: robot kanga_arm, 7 links, 6 joints
Joints:
- joint world_to_link_0: origin xyz=0 0 1.5 rpy=0 0 0 -> xyz=0 0 0.51 rpy=0 0 0

Commit message: joint by joint arm control of the rover

File: kanga_arm/kanga_arm_description/urdf/kanga_arm.urdf (robot description, URDF)
Before this commit: robot kanga_arm, 7 links, 6 joints
Links:
- removed link link_0
- removed link link_1
- removed link link_2
- removed link link_3
- removed link link_4
- removed link link_5
- added link arm_dh_j1, mass 1e-9
- added link arm_dh_j2, mass 1e-9
- added link arm_dh_j3, mass 1e-9
- added link arm_dh_j4, mass 1e-9
- added link arm_dh_j5, mass 1e-9
- added link baserotation, mass 2; collision mesh filename=../meshes/payloads/arm/baserotation.obj; visual mesh filename=../meshes/payloads/arm/baserotation.obj
- added link end_effector_mount, mass 1e-9
- added link gripper_endpoint, mass 1e-9
- added link l4, mass 0.8; collision mesh filename=../meshes/payloads/arm_gripper_payload/l4.obj; visual mesh filename=../meshes/payloads/arm_gripper_payload/l4.obj
- added link l5, mass 0.5; collision mesh filename=../meshes/payloads/arm_gripper_payload/fre_gripper__fixed.o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; collision mesh filename=../meshes/payloads/arm_gripper_payload/l5.obj
- added link link1, mass 2.5; collision mesh filename=../meshes/payloads/arm/link1.obj; visual mesh filename=../meshes/payloads/arm/link1.obj
- added link link2, mass 1; collision mesh filename=../meshes/payloads/arm/link2.obj; visual mesh filename=../meshes/payloads/arm/link2.obj
- added link link3, mass 1; collision mesh filename=../meshes/payloads/arm/link3.obj; visual mesh filename=../meshes/payloads/arm/link3.obj
- added link link4, mass 0.3; collision mesh filename=../meshes/payloads/arm/link4.obj; visual mesh filename=../meshes/payloads/arm/link4.obj
Joints:
- removed joint J1
- removed joint J2
- removed joint J3
- removed joint J4
- removed joint J5
- removed joint world_to_link_0
- added joint arm_dh_j1_frame: type fixed, parent baserotation, child arm_dh_j1, origin xyz=-0.06 0.235 0.006 rpy=0 0 0, axis 0 0 0
- added joint arm_dh_j2_frame: type fixed, parent link1, child arm_dh_j2, origin xyz=0 0 -0.079 rpy=1.5708 -1.05e-10 1.5708, axis 0 0 0
- added joint arm_dh_j3_frame: type fixed, parent link2, child arm_dh_j3, origin xyz=0.449997 1.12725e-06 0.0255 rpy=0 0 -3.14159, axis 0 0 0
- added joint arm_dh_j4_frame: type fixed, parent link4, child arm_dh_j4, origin xyz=0 0 0.0145 rpy=0 0 1.55304, axis 0 0 0
- added joint arm_dh_j5_frame: type fixed, parent l5, child arm_dh_j5, origin xyz=0 0 0.03 rpy=-3.14159 0 0, axis 0 0 0
- added joint arm_gripper_payload_mount_joint: type fixed, parent end_effector_mount, child l4, origin xyz=0 0 0 rpy=0 0 0, axis 0 0 0
- added joint arm_j1: type revolute, parent baserotation, child link1, origin xyz=-0.06 0.235 0.011 rpy=3.14159 0 1.5708, axis 0 0 1, limit lower=-1.5708 upper=1.5708 effort=10 velocity=10
- added joint arm_j2: type revolute, parent link1, child link2, origin xyz=0.0855 5.2029e-07 -0.079 rpy=-6.08527e-06 1.5708 0, axis 0 0 1, limit lower=-1.5708 upper=2.44346 effort=10 velocity=10
- added joint arm_j3: type revolute, parent link2, child link3, origin xyz=0.449997 1.12725e-06 -0.0395 rpy=3.14159 0 0, axis 0 0 1, limit lower=-1.309 upper=2.26893 effort=10 velocity=10
- added joint arm_j4: type revolute, parent link3, child link4, origin xyz=-2.68886e-06 -0.389999 0.04 rpy=-3.14159 0 -3.14159, axis 0 0 1, limit lower=-3.66519 upper=0 effort=10 velocity=10
- added joint arm_j5: type revolute, parent l4, child l5, origin xyz=1.443e-09 -0.03 0.02894 rpy=-1.5708 1.5708 0, axis 0 0 1, limit lower=-3.14159 upper=3.14159 effort=10 velocity=10
- added joint end_effector_mount_frame: type fixed, parent link4, child end_effector_mount, origin xyz=0 0 0.054 rpy=0 0 1.5708, axis 0 0 0
- added joint gripper_endpoint_frame: type fixed, parent l5, child gripper_endpoint, origin xyz=0 -0.0001 -0.211725 rpy=-3.14159 0 2.608e-09, axis 0 0 0
- added joint world_to_baserotation: type fixed, parent world, child baserotation, origin xyz=0 0 2.0 rpy=0 0 0

File: kanga_arm/kanga_arm_description_dep/urdf/kanga_arm.urdf (robot description, URDF)
Before this commit: robot kanga_arm, 7 links, 6 joints
Links:
- link link_0: mass 5 -> 2
- link link_1: mass 5 -> 3
- link link_2: mass 5 -> 3
- link link_3: mass 5 -> 3
- link link_4: mass 5 -> 0.7; geometry collision mesh filename=../meshes/link_4.obj; collision mesh filename=../meshes/realsense_d435.obj
- link link_5: mass 10 -> 0.8
Joints:
- joint J1: limit lower=-1.5708 upper=1.5708 effort=1000 velocity=1000 -> lower=-1.5708 upper=1.5708 effort=100 velocity=100
- joint J2: limit lower=-1.5708 upper=2.44346 effort=1000 velocity=1000 -> lower=-1.5708 upper=2.44346 effort=100 velocity=100; origin xyz=0.0855 -1.39264e-05 -0.056 rpy=-1.5708 -6.12323e-17 1.5708 -> xyz=0.0855 -1.39264e-05 -0.056 rpy=-1.5708 9.90848e-17 1.5708
- joint J3: limit lower=-1.8326 upper=2.87979 effort=1000 velocity=1000 -> lower=-1.8326 upper=2.87979 effort=100 velocity=100; origin xyz=2.76827e-16 0.45 0.0405 rpy=2.51629e-16 -8.53162e-16 -1.77023e-14 -> xyz=-1.5984e-15 0.45 0.0405 rpy=9.42059e-16 3.67644e-15 -2.153e-15
- joint J4: limit lower=-1.309 upper=2.35619 effort=1000 velocity=1000 -> lower=-1.309 upper=2.35619 effort=100 velocity=100; origin xyz=1.04906e-09 0.39 -0.015 rpy=-2.88523e-28 3.54659e-14 1.5708 -> xyz=1.04906e-09 0.39 0.0525 rpy=1.18902e-15 8.86207e-15 1.5708
- joint J5: limit lower=-1.5708 upper=1.5708 effort=1000 velocity=1000 -> lower=-1.5708 upper=1.5708 effort=100 velocity=100; origin xyz=0.105 3.43113e-14 -0.036 rpy=1.5708 3.82745e-33 -1.5708 -> xyz=0.03 1.6784e-14 -0.09644 rpy=3.14159 1.5708 0
- joint world_to_link_0: origin xyz=0 0 0.51 rpy=0 0 0 -> xyz=0 0 1.5 rpy=0 0 0

Commit message: Functional Joint by joint control and ok world space control

File: kanga_arm/kanga_arm_description/urdf/kanga_arm.urdf (robot description, URDF)
Before this commit: robot kanga_arm, 15 links, 14 joints
Joints:
- joint arm_j4: limit lower=-3.66519 upper=0 effort=10 velocity=10 -> lower=-3.66519 upper=0.785398163 effort=10 velocity=10

Commit message: Removed hardware limits in sim, updated the software limits, did some cleanup

File: kanga_arm/kanga_arm_description/urdf/kanga_arm.urdf (robot description, URDF)
Before this commit: robot kanga_arm, 15 links, 14 joints
Joints:
- joint arm_j1: limit lower=-1.5708 upper=1.5708 effort=10 velocity=10 -> lower=-31.4159 upper=31.4159 effort=10 velocity=10
- joint arm_j2: limit lower=-1.5708 upper=2.44346 effort=10 velocity=10 -> lower=-31.4159 upper=31.4159 effort=10 velocity=10
- joint arm_j3: limit lower=-1.309 upper=2.26893 effort=10 velocity=10 -> lower=-31.4159 upper=31.4159 effort=10 velocity=10
- joint arm_j4: limit lower=-3.66519 upper=0.785398163 effort=10 velocity=10 -> lower=-31.4159 upper=31.4159 effort=10 velocity=10
- joint arm_j5: limit lower=-3.14159 upper=3.14159 effort=10 velocity=10 -> lower=-31.4159 upper=31.4159 effort=10 velocity=10
